File: Documentation/420Accumulator/420Accumulator.kicad_sch (KiCad schematic)
At the start: 59 parts, among them J1 AMPSEAL, J2 Conn_01x14, P1 SURLOK, P2 SURLOK, U1 SMD, U2 AIR, U3 AIR, U4 Cell Board, U5 Cell Board

Commit message: post comp
Parts:
- added F1: Fuse, symbol Device:Fuse
Connections:
- net at B75.4 (T-): now also F1.2; no longer U1.
- new net: F1.1, U1.
Other:
- note added: "In"
- note added: "Out of Pack"
- company: (none) -> AERO-SEED
- title: (none) -> Wiring Diagram
