File: PACman LV/IsoSPI.kicad_sch (KiCad schematic)
At the start: 5 parts, among them IC1 LTC6820HMS#3ZZPBF, IC2 LTC6820HMS#3ZZPBF, T1 CoilCraft, T2 CoilCraft

Commit message: post comp
Parts:
- removed IC2: LTC6820HMS#3ZZPBF, SOP50P490X110-16N, symbol AERO:LTC6820HMS#3ZZPBF
- removed T1: CoilCraft, symbol Device:Transformer_1P_1S
- added C1, C2: 0.01u, Capacitor_SMD:C_0603_1608Metric_Pad1.08x0.95mm_HandSolder, symbol Device:C
- added IC1: LTC6820HMS#3ZZPBF, AERO_Footprints:SOP50P490X110-16N, symbol AERO:LTC6820HMS#3ZZPBF
- added JP1, JP2: Fast / Slow, Jumper:SolderJumper-3_P1.3mm_Bridged2Bar12_RoundedPad1.0x1.5mm_NumberLabels, symbol Jumper:Jumper_3_Bridged12
- added R10: 60, Resistor_SMD:R_0603_1608Metric_Pad0.98x0.95mm_HandSolder, symbol Device:R_US
- added R6, R7, R8, R9: 1k, Resistor_SMD:R_0603_1608Metric_Pad0.98x0.95mm_HandSolder, symbol Device:R_US
- added T2: CoilCraft, AERO_Footprints:SRF4532-220Y, symbol Device:Transformer_1P_1S
- IC1: footprint SOP50P490X110-16N -> AERO_Footprints:SOP50P490X110-16N
- R5: footprint (none) -> Resistor_SMD:R_0603_1608Metric_Pad0.98x0.95mm_HandSolder
- T2: footprint (none) -> AERO_Footprints:SRF4532-220Y
Connections:
- net GND: now also IC1.14 (GND), C1.2, C2.2, IC1.1 (EN), IC1.14 (GND), IC1.7 (POL), IC1.8 (PHA), JP1.3 (B), JP2.3 (B), R7.2, R9.2
- net IsoSpi1+: now also T2.4 (SB)
- net IsoSpi1-: now also T2.3 (SA)
- net +3.3V: now reaches IC1.12 (MSTR)
- net +3.3V: now also IC1.6 (VDDS), IC1.7 (POL), IC1.8 (PHA), IC1.9 (VDD), C1.1, C2.1, IC1.12 (MSTR), IC1.6 (VDDS), IC1.9 (VDD), JP1.2 (C), JP2.2 (C)
- net at IC1.13 (SLOW): now also JP1.1 (A)
- net at IC1.15 (ICMP): now also R6.2, R7.1
- net at IC1.16 (IBIAS): now also R6.1
- net MOSI: now reaches IC1.2 (MOSI)
- net MOSI: now also IC1.2 (MOSI)
- net MISO: now reaches IC1.3 (MISO)
- net MISO: now also IC1.3 (MISO)
- net SCK: now reaches IC1.4 (SCK)
- net SCK: now also IC1.4 (SCK)
- net CS2: now reaches IC1.5 (~{CS})
- new net: IC1.11 (IP), R10.1, T2.1 (AA)
- new net: IC1.10 (IM), R10.2, T2.2 (AB)
- new net: IC1.13 (SLOW), JP2.1 (A)
- new net: IC1.15 (ICMP), R8.2, R9.1
- new net: IC1.16 (IBIAS), R8.1
- new net CS1: IC1.5 (~{CS})
