File: PACman LV/PACman LV.kicad_sch (KiCad schematic)
At the start: 19 parts, among them J3 Conn_01x01, J4 Conn_01x01, J5 Conn_01x01, J6 Conn_01x02, J7 Conn_01x14, J9 JST PH, K1 G2RL, K2 G5V-1, K3 G5V-1, Q2 MMBT2222A

Commit message: post comp
Parts:
- removed F3: Fuse, AERO_Footprints:Fuseholder_Blade_Mini_Keystone_3568, symbol Device:Fuse
- added R13, R14: 5k, Resistor_SMD:R_0603_1608Metric_Pad0.98x0.95mm_HandSolder, symbol Device:R_US
- J7: footprint (none) -> AERO_Footprints:TE_1-776266-1_14pin_Horizontal
- R3: value 500 -> 5k; footprint Package_TO_SOT_THT:TO-220-2_Horizontal_TabDown -> Resistor_THT:R_Axial_Power_L48.0mm_W12.5mm_P55.88mm
Connections:
- net FAN_OUT: now also J6.1 (Pin_1)
- net SCK: now also J7.4 (Pin_4); no longer J7.5 (Pin_5)
- net CS renamed CS1
- net CS1: now also R13.2
- new net +3.3V: R13.1, R14.1
- new net CS2: J7.5 (Pin_5), R14.2
Other:
- sheet IsoSpi ports: added CS1, CS2, MISO, MOSI, SCK; removed none
