File: Big Daddy/Big Daddy.kicad_pcb (KiCad board)
At the start: 4 copper layers, 4.1 x 69.3 mm, 109 parts, among them J1 JST-B2B-VERT-2PIN, J10 Conn_01x02, J11 Conn_01x23, J12 Conn_01x14, J13 Conn_01x14, J2 JST-B2B-VERT-2PIN, J3 HV+, J4 HV-, J5 GND, J6 HV+, J7 HV-, J8 Conn_01x14, J9 Conn_01x08, K1 T9VV1K15-12S, K2 G5V-2, K3 G5V-2, K4 J107, K5 G5V-1, Q1 2N7002, Q2 BCP53, U1 MAX33054EASA+T, U10 TLP184, U2 ESP32-S3-DevKitC, U3 ESP32-S3-DevKitC, U4 LT1528CQ#PBF, U5 LTV-817S, U6 ICM7555xB, U7 IS31LT3360, U8 Vicor_AERO, U9 LTV-817S

Commit message: edge cuts
Parts:
- moved K4 20.2 mm to (275.3, 94.3)
- moved C8 20.2 mm to (246.6, 89.2)
- moved D7 20.2 mm to (272.3, 109.0)
- moved K5 20.2 mm to (257.7, 91.4)
- moved F1 20.2 mm to (229.6, 111.3)
- moved F3 20.2 mm to (235.3, 104.1)
- moved F6 20.2 mm to (253.2, 110.8)
- moved F2 20.2 mm to (226.3, 104.1)
- moved C6 20.2 mm to (262.6, 94.3)
- moved C7 20.2 mm to (260.3, 82.2)
- moved D8 20.2 mm to (255.0, 95.8)
- moved F4 20.2 mm to (244.3, 104.1)
- moved F5 20.2 mm to (256.7, 117.5)
- moved D2 19.6 mm to (207.4, 111.0)
- moved K1 19.6 mm to (207.9, 89.0)
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Other:
- board size 4.1 x 69.3 mm -> 298.2 x 125.7 mm

Commit message: Schematic DONE
Parts:
- moved U3 5.19 mm to (358.6, 142.7)
Changed lines of the file:
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@@
   )
   (footprint "esp32:ESP32-S3-DevKitC" (layer "F.Cu")
-    (at 354.53252 145.9162 -90)
+    (at 358.648 142.748 -90)
     (descr "ESP32-S3 general-purpose development board, based on ESP32-S3-WROOM-1 or ESP32-S3-WROOM-1U,It has all the ESP32-S3 pins exposed and is easy to connect and use.")
     (tags "ESP32-S3")
@@
     )
   )
-  (gr_line (start 163.382999 31.852) (end 163.382998 252.577997)
+  (gr_line (start 156.464001 31.496003) (end 156.464 252.222)
     (stroke (width 0.2) (type dot)) (layer "F.SilkS"))
   (gr_line (start 156.209998 152.119) (end 156.209999 101.064999)

Commit message: so cloes
Parts:
- removed R14, R16: 10k, Resistor_SMD:R_0603_1608Metric_Pad0.98x0.95mm_HandSolder
- added C18: C, Capacitor_SMD:C_0603_1608Metric_Pad1.08x0.95mm_HandSolder, B.Cu at (187.3, 87.1)
- added C19: C, Capacitor_SMD:C_0603_1608Metric_Pad1.08x0.95mm_HandSolder, B.Cu at (184.0, 98.0)
- added C20: C, Capacitor_SMD:C_0603_1608Metric_Pad1.08x0.95mm_HandSolder, B.Cu at (164.3, 91.5)
- added D10: SS16, Diode_SMD:D_SMA, F.Cu at (185.8, 77.4)
- added D11: SS16, Diode_SMD:D_SMA, F.Cu at (173.0, 98.0)
- added Q3: IXFH34N65X2, PCM_Package_TO_SOT_THT_AKL:TO-247-3_Vertical_GDS, F.Cu at (175.3, 82.2)
- added Q4: IXFH34N65X2, PCM_Package_TO_SOT_THT_AKL:TO-247-3_Vertical_GDS, F.Cu at (175.4, 91.4)
- added Q6: MMBT2222, Package_TO_SOT_SMD:SOT-23, B.Cu at (168.7, 86.1)
- added R34: .2, Resistor_SMD:R_0805_2012Metric_Pad1.20x1.40mm_HandSolder, B.Cu at (161.3, 79.7)
- added R41: 100, Resistor_SMD:R_0603_1608Metric_Pad0.98x0.95mm_HandSolder, B.Cu at (171.4, 86.1)
- added R42: 2.4k, Resistor_SMD:R_0603_1608Metric_Pad0.98x0.95mm_HandSolder, B.Cu at (164.3, 87.9)
- added R43: 240, Resistor_SMD:R_0603_1608Metric_Pad0.98x0.95mm_HandSolder, B.Cu at (164.3, 84.1)
- added U11: LM5050-1, Package_TO_SOT_SMD:TSOT-23-6, B.Cu at (182.6, 86.9)
- added U12: LM5050-1, Package_TO_SOT_SMD:TSOT-23-6, B.Cu at (180.3, 98.0)
- added U14: LM317_TO-263, Package_TO_SOT_SMD:TO-263-2, B.Cu at (152.8, 88.1)
- C4, C5, C6, C7, D2, D3, D4, D7, Q1, Q2, R1, R12, R13, R15, R17, R18, R19, R2, R20, R21, R22, R23, R28, R3, R31, R39, R4, R5, R6, R7, U4: moved to B.Cu
- J9: footprint AMP_seal:TE_1-776280-1_8pin_Horizontal -> AERO_Footprints:TE_1-776280-1_8pin_Horizontal
- R8: value 330 -> 10k; moved to B.Cu
- R9: value 330 -> 10k
- moved J5 118.6 mm to (152.1, 70.4)
- moved U3 115.6 mm to (245.6, 167.1), turned to 90 degrees
- moved F10 75.7 mm to (189.7, 154.4), turned to -90 degrees
- moved J11 73.3 mm to (262.4, 175.6)
- moved J13 71.8 mm to (220.5, 179.3)
- moved R9 69.7 mm to (284.7, 110.1), turned to 0 degrees
- moved J9 66.6 mm to (174.0, 179.1)
- moved U2 60.1 mm to (245.6, 135.9)
- moved R1 60.1 mm to (253.1, 139.2)
- moved R2 60.0 mm to (255.7, 139.2)
- moved R3 59.9 mm to (258.4, 139.2)
- moved R4 59.9 mm to (261.0, 139.2)
- moved R6 59.5 mm to (283.8, 130.8)
- moved R7 59.5 mm to (286.4, 130.8)
- moved R5 59.5 mm to (281.3, 130.8), turned to -90 degrees
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Connections:
- C10 pad 1: VCC -> VDD
- C17 pad 1: /Connectors/Batt_12 -> /Fusing/Vicor_In
- F9 pad 1: /Connectors/Batt_12 -> /Connectors/Batt_12_IN
- J11 pad 19: /Connectors/BL_TEMP -> /Connectors/BL_STRAIN0
- J11 pad 23: /Connectors/BL_STRAIN0 -> /Connectors/BL_TEMP
- J12 pad 1: /Connectors/RTD_BUZZER_OUT -> /Connectors/CAN_L
- J12 pad 10: /Connectors/DRIVE_MODE_LED -> /Connectors/RTD_BUZZER_OUT
- J12 pad 11: /Connectors/DRIVE_MODE_BTTN -> unconnected-(J12-Pin_11-Pad11)
- J12 pad 12: /Connectors/START_BTTN -> unconnected-(J12-Pin_12-Pad12)
- J12 pad 13: /Connectors/Coast_Regen -> /Connectors/Brake_Regen
- J12 pad 14: /Connectors/Brake_Regen -> /Connectors/Coast_Regen
- J12 pad 2: /Connectors/CAN_L -> /Connectors/CAN_H
- J12 pad 3: /Connectors/CAN_H -> /Connectors/START_BTTN
- J12 pad 4: unconnected-(J12-Pin_4-Pad4) -> /Connectors/DRIVE_MODE_LED
- J12 pad 5: /Connectors/RTD_LED -> /Connectors/DRIVE_MODE_BTTN
- J12 pad 6: /Connectors/FAN_LED -> /Connectors/RTD_LED
- J12 pad 7: /Connectors/PUMP_LED -> unconnected-(J12-Pin_7-Pad7)
- J12 pad 8: /Connectors/IMD_Fault_ind -> /Connectors/BMS_Fault_ind
- J12 pad 9: /Connectors/BMS_Fault_ind -> /Connectors/IMD_Fault_ind
- J8 pad 1: unconnected-(J8-Pin_1-Pad1) -> /Connectors/FAN_PWR_OUT
- J8 pad 10: unconnected-(J8-Pin_10-Pad10) -> /Connectors/BRAKE_PWR_OUT
- J8 pad 11: /Connectors/Batt_12 -> /Connectors/Batt_12_IN
- J8 pad 12: /Connectors/Batt_12 -> /Connectors/Batt_12_IN
- J8 pad 13: /Connectors/Batt_12 -> /Connectors/Batt_12_IN
- J8 pad 14: /Connectors/Batt_12 -> /Connectors/Batt_12_IN
- J8 pad 2: unconnected-(J8-Pin_2-Pad2) -> /Connectors/PUMP_12V
- J8 pad 4: /Connectors/FAN_PWR_OUT -> /Connectors/BMS_12V
- J8 pad 5: /Connectors/BRAKE_PWR_OUT -> /Connectors/RINE_12V
- J8 pad 6: /Connectors/RINE_12V -> /Connectors/FAN_PWR_OUT
- J8 pad 7: /Connectors/BMS_12V -> unconnected-(J8-Pin_7-Pad7)
- J9 pad 1: /Connectors/TSAL_GND -> /Connectors/TSAL_PWR
- J9 pad 2: /Connectors/TSAL_PWR -> /Connectors/TSAL_GND
- J9 pad 3: /Connectors/SSOK -> /Connectors/BRB_LOOP
- J9 pad 5: /Connectors/IMD_FAULT_SIG -> /Connectors/SSOK
- J9 pad 8: /Connectors/BRB_LOOP -> /Connectors/IMD_FAULT_SIG
- K1 pad 3: /Connectors/Batt_12 -> /Fusing/12_prefuse
- L3 pad 2: /Connectors/Batt_12 -> /Fusing/Vicor_In
- R26 pad 2: VCC -> VDD
- R40 pad 1: /Connectors/Batt_12 -> /Fusing/Vicor_In
- R8 pad 1: /Connectors/FAN_LED -> /High Voltage/Vicor_Enable
- R8 pad 2: Net-(U2-GPIO12/ADC2_CH1) -> GND
- R9 pad 1: /Connectors/PUMP_LED -> /Connectors/START_BTTN
- R9 pad 2: Net-(U2-GPIO13/ADC2_CH2) -> GND
- U2 pad 12: unconnected-(U2-GPIO8/ADC1_CH7-Pad12) -> /Microcontrolller/Traction_Toggle
- U2 pad 18: Net-(U2-GPIO12/ADC2_CH1) -> /High Voltage/Vicor_Fault
- U2 pad 19: Net-(U2-GPIO13/ADC2_CH2) -> /High Voltage/Vicor_Enable
- U2 pad 20: /Microcontrolller/VICOR_Tempt? -> /Microcontrolller/RTD_BUZZER
- U2 pad 25: unconnected-(U2-GPIO19/USB_D--Pad25) -> /Connectors/BL_SPEED
- U2 pad 26: unconnected-(U2-GPIO20/USB_D+-Pad26) -> /Connectors/BR_SPEED
- U2 pad 27: /High Voltage/Vicor_Fault -> /Connectors/FL_SPEED
- U2 pad 28: /High Voltage/Vicor_Enable -> /Connectors/FR_SPEED
- U2 pad 29: /Microcontrolller/RTD_BUZZER -> /Connectors/START_BTTN
- U2 pad 32: /Connectors/START_BTTN -> /Microcontrolller/SCL
- U2 pad 33: unconnected-(U2-GPIO36-Pad33) -> /Microcontrolller/SDA
- U2 pad 34: /Cooling/Fan_SIG_Out -> /Cooling/Brake_SIG_Out
- U2 pad 35: /Cooling/Brake_SIG_Out -> /Cooling/Fan_SIG_Out
- U2 pad 8: /Latching/IMD_IND -> /Latching/BMS_IND
- U2 pad 9: /Latching/BMS_IND -> /Latching/IMD_IND
- U3 pad 10: /Connectors/FL_SPEED -> unconnected-(U3-GPIO17/ADC2_CH6-Pad10)
- U3 pad 38: /Connectors/BL_SPEED -> unconnected-(U3-GPIO41/MTDI-Pad38)
- U3 pad 39: /Connectors/BR_SPEED -> unconnected-(U3-GPIO42/MTMS-Pad39)
- U3 pad 42: unconnected-(U3-GPIO44/U0RXD-Pad42) -> /Microcontrolller/Core_RX
- U3 pad 43: unconnected-(U3-GPIO43/U0TXD-Pad43) -> /Microcontrolller/Core_TX
- U3 pad 5: /Connectors/FR_SPEED -> unconnected-(U3-GPIO5/ADC1_CH4-Pad5)
- U5 pad 4: VCC -> VDD
- U6 pad 8: VCC -> VDD
Routing:
- net /High Voltage/Vicor_Fault: track 0.00 -> 189.6 mm, vias 0 -> 1
- net VDD: track 0.00 -> 185.4 mm, vias 0 -> 5
- net GND: track 0.00 -> 170.4 mm, vias 0 -> 45
- net /High Voltage/Vicor_Enable: track 0.00 -> 156.2 mm
- net INT_12V: track 0.00 -> 110.3 mm, vias 0 -> 6
- net /Connectors/Batt_12_IN: track 0.00 -> 86.1 mm
- net /Connectors/Brake_Regen: track 0.00 -> 82.0 mm, vias 0 -> 1
- net /Connectors/Coast_Regen: track 0.00 -> 80.3 mm, vias 0 -> 1
- net /Connectors/BRB_RTN: track 0.00 -> 79.0 mm
- net /Connectors/IMD_Fault_ind: track 0.00 -> 75.1 mm
- net /Connectors/BMS_FAULT_SIG: track 0.00 -> 73.7 mm
- net /Connectors/RTD_BUZZER_OUT: track 0.00 -> 69.6 mm
- net /Connectors/RTD_LED: track 0.00 -> 67.9 mm
- net /Latching/BMS_IND: track 0.00 -> 66.6 mm
- net /Connectors/BMS_Fault_ind: track 0.00 -> 64.9 mm
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- added copper zone on B.Cu, net +12V
- added copper zone on F.Cu, net +12V
- added copper zone on B.Cu, net /Connectors/BMS_12V
- added copper zone on F.Cu, net /Connectors/BMS_12V
- added copper zone on B.Cu, net /Connectors/BRAKE_PWR_OUT
- added copper zone on F.Cu, net /Connectors/BRAKE_PWR_OUT
- added copper zone on B.Cu, net /Connectors/Batt_12_IN
- added copper zone on F.Cu, net /Connectors/Batt_12_IN
- added copper zone on B.Cu, net /Connectors/FAN_PWR_OUT
- added copper zone on F.Cu, net /Connectors/FAN_PWR_OUT
- added copper zone on B.Cu, net /Connectors/PUMP_12V
- added copper zone on F.Cu, net /Connectors/PUMP_12V
- added copper zone on B.Cu, net /Connectors/RINE_12V
- added copper zone on F.Cu, net /Connectors/RINE_12V
- added copper zone on B.Cu, net /Cooling/BRAKE_12V
- added copper zone on F.Cu, net /Cooling/BRAKE_12V
- added copper zone on B.Cu, net /Cooling/FAN_12V
- added copper zone on F.Cu, net /Cooling/FAN_12V
- added copper zone on B.Cu, net /Fusing/12_prefuse
- added copper zone on F.Cu, net /Fusing/12_prefuse
- added copper zone on B.Cu, net /Fusing/Vicor_In
- added copper zone on F.Cu, net /Fusing/Vicor_In
- added copper zone on F.Cu, net /High Voltage/DCDC/HV+
- added copper zone on F.Cu, net /High Voltage/DCDC/HV-
- added copper zone on F.Cu, net /High Voltage/TSAL/HV+
- added copper zone on In2.Cu, net GND
- added copper zone on In1.Cu, net INT_12V
- added copper zone on B.Cu, net Net-(J6-Pin_1)
- added copper zone on F.Cu, net Net-(J6-Pin_1)
- added copper zone on B.Cu, net Net-(J7-Pin_1)
- added copper zone on F.Cu, net Net-(J7-Pin_1)
- added copper zone on F.Cu, net Net-(U8-+IN)
- added copper zone on B.Cu, net Net-(U8-+OUT)
- added copper zone on F.Cu, net Net-(U8-+OUT)
- added copper zone on In1.Cu, net VDD
Other:
- board size 298.2 x 125.7 mm -> 245.1 x 127 mm
- board text added: "locked"
- board text removed: "HV!"
- board text removed: "LV"
- board text removed: "{dblquote}HV Board{dblquote}"

Commit message: REVIEW TIME
Connections:
- J11 pad 1: unconnected-(J11-Pin_1-Pad1) -> /Connectors/FR_STRAIN1
- J11 pad 10: /Connectors/FL_TEMP -> /Connectors/FL_STRAIN0
- J11 pad 11: /Connectors/FL_SPEED -> /Connectors/RPi_TX
- J11 pad 12: /Connectors/FL_STRAIN0 -> /Connectors/RPi_RX
- J11 pad 13: /Connectors/FL_STRAIN1 -> /Connectors/BR_STRAIN1
- J11 pad 14: /Connectors/BR_SUS -> /Connectors/FR_TEMP
- J11 pad 15: /Connectors/BR_TEMP -> /Connectors/FL_SPEED
- J11 pad 16: /Connectors/BR_STRAIN0 -> /Connectors/FR_SUS
- J11 pad 17: /Connectors/BR_STRAIN1 -> /Connectors/FL_SUS
- J11 pad 18: /Connectors/BL_SUS -> /Connectors/FL_STRAIN1
- J11 pad 19: /Connectors/BL_STRAIN0 -> /Connectors/BR_STRAIN0
- J11 pad 2: /Connectors/FBrake -> /Connectors/FL_TEMP
- J11 pad 20: /Connectors/BL_SPEED -> unconnected-(J11-Pin_20-Pad20)
- J11 pad 21: /Connectors/BR_SPEED -> /Connectors/FR_SPEED
- J11 pad 22: /Connectors/BL_STRAIN1 -> /Connectors/BR_SPEED
- J11 pad 23: /Connectors/BL_TEMP -> /Connectors/BL_SPEED
- J11 pad 3: /Connectors/RBrake -> unconnected-(J11-Pin_3-Pad3)
- J11 pad 4: /Connectors/FR_TEMP -> /Connectors/BR_SUS
- J11 pad 5: /Connectors/FR_SUS -> /Connectors/BR_TEMP
- J11 pad 6: /Connectors/FR_SPEED -> /Connectors/STEERING
- J11 pad 7: /Connectors/FR_STRAIN0 -> /Connectors/BL_SUS
- J11 pad 8: /Connectors/FR_STRAIN1 -> /Connectors/BL_TEMP
- J11 pad 9: /Connectors/FL_SUS -> /Connectors/FR_STRAIN0
- J13 pad 1: unconnected-(J13-Pin_1-Pad1) -> /Connectors/PUMP_TEMP_IN
- J13 pad 10: /Connectors/GPS_RX -> /Connectors/Pedal_1
- J13 pad 11: /Connectors/GPS_TX -> /Connectors/BL_STRAIN0
- J13 pad 12: /Connectors/STEERING -> /Connectors/GPS_RX
- J13 pad 13: /Connectors/PUMP_TEMP_OUT -> /Connectors/LoRa_TX
- J13 pad 14: /Connectors/PUMP_TEMP_IN -> /Connectors/LoRa_RX
- J13 pad 3: /Connectors/Pedal_1 -> /Connectors/FBrake
- J13 pad 4: /Connectors/RPi_RX -> /Connectors/BL_STRAIN1
- J13 pad 5: /Connectors/RPi_TX -> /Connectors/IMU_TX
- J13 pad 6: /Connectors/LoRa_RX -> /Connectors/PUMP_TEMP_OUT
- J13 pad 7: /Connectors/LoRa_TX -> /Connectors/RBrake
- J13 pad 8: /Connectors/IMU_RX -> /Connectors/GPS_TX
- J13 pad 9: /Connectors/IMU_TX -> /Connectors/IMU_RX
Routing:
- net /Connectors/BR_SPEED: track 0.00 -> 82.8 mm
- net /Connectors/BL_SPEED: track 0.00 -> 80.7 mm
- net /Connectors/PUMP_TEMP_IN: track 0.00 -> 79.2 mm, vias 0 -> 1
- net /Connectors/FL_SPEED: track 0.74 -> 77.4 mm
- net /Connectors/FR_SPEED: track 1.22 -> 77.2 mm
- net /Connectors/Pedal_1: track 4.40 -> 74.1 mm
- net /Connectors/RBrake: track 3.86 -> 71.1 mm
- net /Connectors/LoRa_RX: track 0.00 -> 66.2 mm
- net /Connectors/LoRa_TX: track 0.42 -> 65.4 mm
- net /Connectors/GPS_RX: track 0.00 -> 63.7 mm
- net /Connectors/IMU_RX: track 0.41 -> 61.9 mm
- net /Connectors/FBrake: track 2.44 -> 63.2 mm
- net /Connectors/GPS_TX: track 0.32 -> 57.4 mm
- net /Connectors/Pedal_0: track 5.38 -> 61.3 mm
- net /Connectors/BL_STRAIN0: track 0.28 -> 55.2 mm
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Other:
- board size 245.1 x 127 mm -> 245.5 x 127 mm
- board text added: "HV!"
- board text added: "LV"
- board text added: "{dblquote}HV Board{dblquote}"
- board text removed: "locked"

Commit message: updates
Parts:
- added F7: 2A, AERO_Footprints:Fuseholder_Blade_Mini_Keystone_3568, F.Cu at (223.1, 122.5)
- added G***: LOGO, AERO_Footprints:hvlightningsymbol, F.Cu at (69.5, 123.5)
- added G***: LOGO, AERO_Footprints:AERO_Logo_15x6mm, F.Cu at (154.0, 74.5)
- added G***: LOGO, AERO_Footprints:Bessie_10x10, F.Cu at (154.0, 83.0)
- added J15: Conn_01x02, AERO_Footprints:TE_MATE-N-LOK_1-770866-x_1x02_P4.14mm_Vertical, F.Cu at (174.2, 67.8)
- moved J5 97.3 mm to (154.5, 167.7)
Connections:
- J11 pad 20: unconnected-(J11-Pin_20-Pad20) -> GND
- J11 pad 3: unconnected-(J11-Pin_3-Pad3) -> GND
- J12 pad 11: unconnected-(J12-Pin_11-Pad11) -> GND
- J12 pad 12: unconnected-(J12-Pin_12-Pad12) -> GND
- J12 pad 7: unconnected-(J12-Pin_7-Pad7) -> GND
- J8 pad 1: /Connectors/FAN_PWR_OUT -> /Connectors/BMS_FAN_PWR_OUT
- J8 pad 7: unconnected-(J8-Pin_7-Pad7) -> GND
- J8 pad 8: unconnected-(J8-Pin_8-Pad8) -> GND
- J8 pad 9: unconnected-(J8-Pin_9-Pad9) -> GND
Routing:
- net /Connectors/BMS_FAN_PWR_OUT: track 0.00 -> 61.9 mm
- net /High Voltage/Vicor_Fault: track 189.6 -> 158.1 mm, vias 1 -> 3
Other:
- board text added: "12v -> 3v"
- board text added: "BMS"
- board text added: "BMS FAN"
- board text added: "BRAKE"
- board text added: "BRB"
- board text added: "CAN"
- board text added: "CAN / DASH"
- board text added: "CAN_H"
- board text added: "CAN_L"
- board text added: "DAQ"
- board text added: "FAN"
- board text added: "GND"
- board text added: "HV+ IN"
- board text added: "HV+ Test"
- board text added: "HV- IN"
- board text added: "HV- Test"
- board text added: "IMD"
- board text added: "INTERNAL"
- board text added: "Main Board V1 C.Grund 39-24"
- board text added: "OTHER SENSORS"
- board text added: "POWER"
- board text added: "PUMP"
- board text added: "RINEHART"
- board text added: "SAFTEY"
- board text added: "SSOK"
- board text added: "Saftey Loop"
- board text added: "Tractive"
- board text added: "WHEELS"
- board text added: "{dblquote}Fusing{dblquote}"

Commit message: Updated BOM
Parts:
- J1: value JST-B2B-VERT-2PIN -> BMS Button
- J2: value JST-B2B-VERT-2PIN -> IMD Button
- R32: value 10k -> 20k; footprint Resistor_THT:R_Axial_Power_L50.0mm_W9.0mm_P60.96mm -> Resistor_THT:R_Axial_DIN0309_L9.0mm_D3.2mm_P5.08mm_Vertical
- R33: value 10k -> 20K; footprint Resistor_THT:R_Axial_Power_L50.0mm_W9.0mm_P60.96mm -> Resistor_THT:R_Axial_DIN0309_L9.0mm_D3.2mm_P5.08mm_Vertical
- moved R32 30.3 mm to (94.9, 93.0)
- moved R33 24.6 mm to (90.9, 165.0)
- moved J13 0.83 mm to (220.5, 178.5)
Connections:
- R42 pad 2: Net-(Q6-C) -> Net-(U14-ADJ)
- R43 pad 1: Net-(Q6-C) -> Net-(U14-ADJ)
- U14 pad 1: Net-(Q6-C) -> Net-(U14-ADJ)
