File: Big Daddy/Big Daddy.kicad_sch (KiCad schematic)
At the start: 0 parts

Commit message: George Redlines for Big Daddy board
Other:
- note added: "General Notes: - Suggest putting part numbers for each part in the properties. When exporting the BOM, all part numbers are there -- then can import to DigiKey or others"
Changed lines of the file:
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@@
     (stroke (width 0) (type default))
+  )
+  (text "General Notes: \n- Suggest putting part numbers for each part in the properties.\nWhen exporting the BOM, all part numbers are there -- then can import to DigiKey or others"
+    (at 21.59 182.88 0)
+    (effects (font (size 1.27 1.27) (color 255 7 28 1)) (justify left bottom))
   )
   (global_label "INT_12V" (shape input) (at 92.964 20.828 0) (fields_autoplaced)
