File: Big Daddy/Big Daddy.kicad_sch (KiCad schematic)
At the start: 0 parts

Commit message: so cloes
Other:
- sheet Connectors ports: added Batt_12_IN; removed Batt_12, VICOR_Tempt?
- sheet Fusing ports: added Batt_12_IN, Vicor_In; removed Batt_12
Changed lines of the file:
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@@
   (junction (at 94.488 80.264) (diameter 0) (color 0 0 0 0)
   )
-  (junction (at 39.37 66.548) (diameter 0) (color 0 0 0 0)
-  )
   (wire (pts (xy 39.37 136.398) (xy 51.816 136.398))
     (stroke (width 0) (type default))
@@
     (stroke (width 0) (type default))
   )
-  (wire (pts (xy 39.37 58.674) (xy 39.37 66.548))
-    (stroke (width 0) (type default))
-  )
   (wire (pts (xy 74.93 20.828) (xy 92.964 20.828))
     (stroke (width 0) (type default))
@@
     (stroke (width 0) (type default))
   )
+  (wire (pts (xy 39.37 136.398) (xy 39.37 83.312))
+    (stroke (width 0) (type default))
+  )
   (wire (pts (xy 146.05 95.758) (xy 190.754 95.758))
     (stroke (width 0) (type default))
@@
     (stroke (width 0) (type default))
   )
+  (wire (pts (xy 56.134 81.026) (xy 39.37 81.026))
+    (stroke (width 0) (type default))
+  )
   (wire (pts (xy 75.692 135.89) (xy 112.776 135.89))
     (stroke (width 0) (type default))
@@
     (stroke (width 0) (type default))
   )
-  (wire (pts (xy 39.37 66.548) (xy 39.37 136.398))
-    (stroke (width 0) (type default))
-  )
   (wire (pts (xy 146.05 50.546) (xy 190.754 50.546))
     (stroke (width 0) (type default))
@@
     (stroke (width 0) (type default))
   )
+  (wire (pts (xy 39.37 83.312) (xy 56.134 83.312))
+    (stroke (width 0) (type default))
+  )
+  (wire (pts (xy 39.37 81.026) (xy 39.37 58.674))
+    (stroke (width 0) (type default))
+  )
   (wire (pts (xy 146.05 53.594) (xy 190.754 53.594))
     (stroke (width 0) (type default))
@@
   )
   (wire (pts (xy 146.05 91.186) (xy 190.754 91.186))
-    (stroke (width 0) (type default))
-  )
-  (wire (pts (xy 56.134 66.548) (xy 39.37 66.548))
     (stroke (width 0) (type default))
   )
@@
       (effects (font (size 1.27 1.27)) (justify right))
     )
-    (pin "VICOR_Tempt?" input (at 146.05 104.648 0)
-      (effects (font (size 1.27 1.27)) (justify right))
-    )
     (pin "Coast_Regen" input (at 146.05 101.346 0)
       (effects (font (size 1.27 1.27)) (justify right))
@@
       (effects (font (size 1.27 1.27)) (justify left))
     )
-    (pin "Batt_12" input (at 112.776 58.674 180)
-      (effects (font (size 1.27 1.27)) (justify left))
-    )
     (pin "IMD_FAULT_SIG" input (at 112.776 30.734 180)
       (effects (font (size 1.27 1.27)) (justify left))
@@
     (pin "PUMP_12V" output (at 146.05 139.446 0)
       (effects (font (size 1.27 1.27)) (justify right))
+    )
+    (pin "Batt_12_IN" input (at 112.776 58.674 180)
+      (effects (font (size 1.27 1.27)) (justify left))
     )
     (instances
@@
       (effects (font (size 1.27 1.27)) (justify right))
     )
-    (pin "Batt_12" input (at 56.134 66.548 180)
-      (effects (font (size 1.27 1.27)) (justify left))
-    )
     (pin "BRB_RTN" input (at 75.692 69.85 0)
       (effects (font (size 1.27 1.27)) (justify right))
@@
       (effects (font (size 1.27 1.27)) (justify right))
     )
+    (pin "Batt_12_IN" input (at 56.134 81.026 180)
+      (effects (font (size 1.27 1.27)) (justify left))
+    )
+    (pin "Vicor_In" input (at 56.134 83.312 180)
+      (effects (font (size 1.27 1.27)) (justify left))
+    )
     (instances

Commit message: updates
Other:
- sheet Connectors ports: added BMS_FAN_PWR_OUT; removed none
- sheet Fusing ports: added PAC_FAN; removed none
Changed lines of the file:
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@@
+    (stroke (width 0) (type default))
+  )
+  (wire (pts (xy 75.692 97.536) (xy 112.776 97.536))
     (stroke (width 0) (type default))
   )
@@
       (effects (font (size 1.27 1.27)) (justify left))
     )
+    (pin "BMS_FAN_PWR_OUT" output (at 112.776 97.536 180)
+      (effects (font (size 1.27 1.27)) (justify left))
+    )
     (instances
       (project "Big Daddy"
@@
       (effects (font (size 1.27 1.27)) (justify left))
     )
+    (pin "PAC_FAN" output (at 75.692 97.536 0)
+      (effects (font (size 1.27 1.27)) (justify right))
+    )
     (instances

Commit message: post comp
Other:
- title: DADDY BOARD -> MAIN LV BOARD
Changed lines of the file:
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@@
   (paper "A")
   (title_block
-    (title "DADDY BOARD")
+    (title "MAIN LV BOARD")
     (date "2023-05-15")
     (rev "V 1.1")
@@
     (stroke (width 0) (type default))
   )
-  (wire (pts (xy 146.05 104.648) (xy 190.754 104.648))
-    (stroke (width 0) (type default))
-  )
