File: Big Daddy/Cooling.kicad_sch (KiCad schematic)
At the start: 7 parts, among them K4 J107, K5 G5V-1

Commit message: George Redlines for Big Daddy board
Other:
- note added: "For the radiator fan, does that have variable speed control? Instead of "on/off", maybe a motor speed control? That would help with startup current. Consider H-Bridge motor driver."
- note added: "The Brake will switch on / off frequently. Consider either PMOS or NMOS "switch" instead of relay. Low(ish) current, so mosfet switch would work fine."
Changed lines of the file:
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@@
     (stroke (width 0) (type default))
+  )
+  (text "For the radiator fan, does that have variable\nspeed control? Instead of \"on/off\", maybe a \nmotor speed control? That would help with startup\ncurrent. Consider H-Bridge motor driver. "
+    (at 39.37 54.61 0)
+    (effects (font (size 1.27 1.27) (color 255 8 38 1)) (justify left bottom))
   )
   (text "Brake" (at 137.16 63.5 0)
@@
     (effects (font (size 3 3)) (justify left bottom))
   )
+  (text "The Brake will switch on / off frequently.\nConsider either PMOS or NMOS \"switch\" instead of relay.\nLow(ish) current, so mosfet switch would work fine. "
+    (at 116.84 50.8 0)
+    (effects (font (size 1.27 1.27) (color 255 0 51 1)) (justify left bottom))
+  )
   (text "Pump" (at 211.836 64.262 0)
