File: Big Daddy/Cooling.kicad_sch (KiCad schematic)
At the start: 7 parts, among them K4 J107, K5 G5V-1

Commit message: Updated BOM
Parts:
- C6, C7, C8: value 10u -> 10uF; Digikey part number (none) -> 1276-1038-1-ND; Manufacturer_Part_Number (none) -> CL10A106KQ8NNNC
- D7, D8: Digikey part number (none) -> 1655-1N4148WCT-ND; Manufacturer_Part_Number (none) -> 1N4148W
