File: Big Daddy/Fusing.kicad_sch (KiCad schematic)
At the start: 24 parts, among them K1 T9VV1K15-12S, Q3 IXFH34N65X2, Q4 IXFH34N65X2, U11 LM5050-1, U12 LM5050-1, U4 LT1528CQ#PBF

Commit message: Schematic DONE
Parts:
- added C20: C, symbol Device:C
- added Q5: 2N2222, Package_TO_SOT_THT_AKL:TO-18-3_EBC, symbol PCM_Transistor_BJT_AKL:2N2222
- added R34: .2, symbol Device:R_US
- added R41: 100, symbol Device:R_US
- added R42: 2.4k, symbol Device:R_US
- added R43: 240, symbol Device:R_US
- added U13: LM317_TO-220, Package_TO_SOT_THT:TO-220-3_Vertical, symbol Regulator_Linear:LM317_TO-220
Connections:
- net Batt_12_IN: now also R34.1, R43.2
- net GND: now also C20.2, Q5.1 (E), R41.2, R42.1
- net Vicor_In: now also C20.1, U13.3 (VI)
- new net: Q5.3 (C), R42.2, R43.1, U13.1 (ADJ)
- new net: R34.2, U13.2 (VO)
- new net: Q5.2 (B), R41.1
Other:
- note added: "Charger For Vicor to Battery"
- moved on the sheet: C18, C19, C4, C5, D10, D11, D2, D3, D4, F1, F10, F2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

Commit message: so cloes
Parts:
- removed Q5: 2N2222, Package_TO_SOT_THT_AKL:TO-18-3_EBC, symbol PCM_Transistor_BJT_AKL:2N2222
- removed U13: LM317_TO-220, Package_TO_SOT_THT:TO-220-3_Vertical, symbol Regulator_Linear:LM317_TO-220
- added Q6: MMBT2222, Package_TO_SOT_SMD:SOT-23, symbol PCM_Transistor_BJT_AKL:MMBT2222
- added U14: LM317_TO-263, Package_TO_SOT_SMD:TO-263-2, symbol Regulator_Linear:LM317_TO-263
- C18, C19, C20: footprint (none) -> Capacitor_SMD:C_0603_1608Metric_Pad1.08x0.95mm_HandSolder
- D10, D11: footprint Diode_SMD_AKL:D_SMA -> Diode_SMD:D_SMA
- Q3, Q4: footprint Package_TO_SOT_THT_AKL:TO-247-3_Vertical_GDS -> PCM_Package_TO_SOT_THT_AKL:TO-247-3_Vertical_GDS
- R34: footprint (none) -> Resistor_SMD:R_0805_2012Metric_Pad1.20x1.40mm_HandSolder
- R41, R42, R43: footprint (none) -> Resistor_SMD:R_0603_1608Metric_Pad0.98x0.95mm_HandSolder
Connections:
- net Batt_12_IN: now also F9.1
- net GND: now also Q6.2 (E)
- net Vicor_In: now also U14.3 (VI)
- net at R42.2, R43.1: now also Q6.3 (C), U14.1 (ADJ)
- net at R34.2: now also U14.2 (VO)
- net at R41.1: now also Q6.1 (B)
- net Batt_12 renamed 12_prefuse
- net 12_prefuse: no longer F9.1
Other:
- moved on the sheet: D11

Commit message: updates
Parts:
- added F7: 2A, AERO_Footprints:Fuseholder_Blade_Mini_Keystone_3568, symbol Device:Fuse
Connections:
- net +12V: now also F7.1
- new net PAC_FAN: F7.2
Other:
- moved on the sheet: F10, F9
Changed lines of the file:
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@@
   (junction (at 78.994 139.7) (diameter 0) (color 0 0 0 0)
+  )
+  (junction (at 203.2 72.644) (diameter 0) (color 0 0 0 0)
   )
   (junction (at 116.586 129.794) (diameter 0) (color 0 0 0 0)
@@
     (stroke (width 0) (type default))
   )
-  (wire (pts (xy 230.632 81.026) (xy 221.488 81.026))
+  (wire (pts (xy 233.172 87.884) (xy 224.028 87.884))
     (stroke (width 0) (type default))
   )
@@
     (stroke (width 0) (type default))
   )
+  (wire (pts (xy 203.2 78.994) (xy 203.2 72.644))
+    (stroke (width 0) (type default))
+  )
   (wire (pts (xy 189.992 140.462) (xy 218.44 140.462))
     (stroke (width 0) (type default))
   )
-  (polyline (pts (xy 190.5 94.742) (xy 248.92 94.996))
+  (polyline (pts (xy 190.246 99.822) (xy 248.666 100.076))
     (stroke (width 0) (type default))
   )
@@
     (stroke (width 0) (type default))
   )
-  (wire (pts (xy 205.74 81.026) (xy 213.868 81.026))
+  (wire (pts (xy 208.28 87.884) (xy 216.408 87.884))
     (stroke (width 0) (type default))
   )
@@
     (stroke (width 0) (type default))
   )
+  (wire (pts (xy 203.2 78.994) (xy 208.534 78.994))
+    (stroke (width 0) (type default))
+  )
   (wire (pts (xy 102.616 94.488) (xy 102.616 115.824))
     (stroke (width 0) (type default))
@@
     (stroke (width 0) (type default))
   )
-  (wire (pts (xy 213.868 88.646) (xy 206.502 88.646))
+  (wire (pts (xy 216.408 95.504) (xy 209.042 95.504))
     (stroke (width 0) (type default))
   )
@@
     (stroke (width 0) (type default))
   )
+  (wire (pts (xy 216.154 78.994) (xy 230.124 78.994))
+    (stroke (width 0) (type default))
+  )
   (wire (pts (xy 122.428 167.64) (xy 115.824 167.64))
     (stroke (width 0) (type default))
@@
     (stroke (width 0) (type default))
   )
-  (wire (pts (xy 230.378 88.646) (xy 221.488 88.646))
+  (wire (pts (xy 232.918 95.504) (xy 224.028 95.504))
     (stroke (width 0) (type default))
   )
@@
     (effects (font (size 1.27 1.27)) (justify right))
   )
-  (hierarchical_label "BRB_LOOP" (shape output) (at 230.632 81.026 0) (fields_autoplaced)
+  (hierarchical_label "BRB_LOOP" (shape output) (at 233.172 87.884 0) (fields_autoplaced)
     (effects (font (size 1.27 1.27)) (justify left))
   )
-  (hierarchical_label "Batt_12_IN" (shape input) (at 205.74 81.026 180) (fields_autoplaced)
+  (hierarchical_label "Batt_12_IN" (shape input) (at 208.28 87.884 180) (fields_autoplaced)
     (effects (font (size 1.27 1.27)) (justify right))
   )
-  (hierarchical_label "LOOP_OUT" (shape input) (at 206.502 88.646 180) (fields_autoplaced)
+  (hierarchical_label "LOOP_OUT" (shape input) (at 209.042 95.504 180) (fields_autoplaced)
     (effects (font (size 1.27 1.27)) (justify right))
   )
-  (hierarchical_label "TSV" (shape output) (at 230.378 88.646 0) (fields_autoplaced)
+  (hierarchical_label "TSV" (shape output) (at 232.918 95.504 0) (fields_autoplaced)
     (effects (font (size 1.27 1.27)) (justify left))
   )
@@
   )
   (hierarchical_label "BRAKE_12V" (shape output) (at 229.87 72.644 0) (fields_autoplaced)
+    (effects (font (size 1.27 1.27)) (justify left))
+  )
+  (hierarchical_label "PAC_FAN" (shape output) (at 230.124 78.994 0) (fields_autoplaced)
     (effects (font (size 1.27 1.27)) (justify left))
   )
@@
     )
   )
-  (symbol (lib_id "Device:Fuse") (at 217.678 88.646 90) (mirror x) (unit 1)
-    (in_bom yes) (on_board yes) (dnp no)
-    (property "Reference" "F10" (at 220.218 86.106 90)
-      (effects (font (size 1.27 1.27)))
-    )
-    (property "Value" "1A" (at 215.138 86.106 90)
-      (effects (font (size 1.27 1.27)))
-    )
-    (property "Footprint" "AERO_Footprints:Fuseholder_Blade_Mini_Keystone_3568" (at 217.678 86.868 90)
-      (effects (font (size 1.27 1.27)) hide)
-    )
-    (property "Datasheet" "~" (at 217.678 88.646 0)
+  (symbol (lib_id "Device:Fuse") (at 220.218 95.504 90) (mirror x) (unit 1)
+    (in_bom yes) (on_board yes) (dnp no)
+    (property "Reference" "F10" (at 222.758 92.964 90)
+      (effects (font (size 1.27 1.27)))
+    )
+    (property "Value" "1A" (at 217.678 92.964 90)
+      (effects (font (size 1.27 1.27)))
+    )
+    (property "Footprint" "AERO_Footprints:Fuseholder_Blade_Mini_Keystone_3568" (at 220.218 93.726 90)
+      (effects (font (size 1.27 1.27)) hide)
+    )
+    (property "Datasheet" "~" (at 220.218 95.504 0)
       (effects (font (size 1.27 1.27)) hide)
     )
@@
         (path "/e63e39d7-6ac0-4ffd-8aa3-1841a4541b55/9c1412ff-15e3-4ef7-9c9c-e6f8f725cc08"
           (reference "U14") (unit 1)
+        )
+      )
+    )
+  )
+  (symbol (lib_id "Device:Fuse") (at 212.344 78.994 90) (mirror x) (unit 1)
+    (in_bom yes) (on_board yes) (dnp no)
+    (property "Reference" "F7" (at 214.884 76.454 90)
+      (effects (font (size 1.27 1.27)))
+    )
+    (property "Value" "2A" (at 209.804 76.454 90)
+      (effects (font (size 1.27 1.27)))
+    )
+    (property "Footprint" "AERO_Footprints:Fuseholder_Blade_Mini_Keystone_3568" (at 212.344 77.216 90)
+      (effects (font (size 1.27 1.27)) hide)
+    )
+    (property "Datasheet" "~" (at 212.344 78.994 0)
+      (effects (font (size 1.27 1.27)) hide)
+    )
+    (pin "1")
+    (pin "2")
+    (instances
+      (project "Big Daddy"
+        (path "/e63e39d7-6ac0-4ffd-8aa3-1841a4541b55/9c1412ff-15e3-4ef7-9c9c-e6f8f725cc08"
+          (reference "F7") (unit 1)
         )
       )
@@
     )
   )
-  (symbol (lib_id "Device:Fuse") (at 217.678 81.026 90) (mirror x) (unit 1)
-    (in_bom yes) (on_board yes) (dnp no)
-    (property "Reference" "F9" (at 220.218 78.486 90)
-      (effects (font (size 1.27 1.27)))
-    )
-    (property "Value" "1A" (at 215.138 78.486 90)
-      (effects (font (size 1.27 1.27)))
-    )
-    (property "Footprint" "AERO_Footprints:Fuseholder_Blade_Mini_Keystone_3568" (at 217.678 79.248 90)
-      (effects (font (size 1.27 1.27)) hide)
-    )
-    (property "Datasheet" "~" (at 217.678 81.026 0)
-      (effects (font (size 1.27 1.27)) hide)
-    )
+  (symbol (lib_id "Device:Fuse") (at 220.218 87.884 90) (mirror x) (unit 1)
+    (in_bom yes) (on_board yes) (dnp no)
+    (property "Reference" "F9" (at 222.758 85.344 90)
+      (effects (font (size 1.27 1.27)))
+    )
+    (property "Value" "1A" (at 217.678 85.344 90)
+      (effects (font (size 1.27 1.27)))
+    )
+    (property "Footprint" "AERO_Footprints:Fuseholder_Blade_Mini_Keystone_3568" (at 220.218 86.106 90)
+      (effects (font (size 1.27 1.27)) hide)
+    )
+    (property "Datasheet" "~" (at 220.218 87.884 0)
+      (effects (font (size 1.27 1.27)) hide)
+    )

Commit message: post comp
Parts:
- removed Q6: MMBT2222, Package_TO_SOT_SMD:SOT-23, symbol PCM_Transistor_BJT_AKL:MMBT2222
- removed R41: 100, Resistor_SMD:R_0603_1608Metric_Pad0.98x0.95mm_HandSolder, symbol Device:R_US
Connections:
- net 12_prefuse: now also Q3.2 (D), Q4.2 (D); no longer Q3.3 (S), Q4.3 (S)
- net Batt_12_IN: now also Q3.3 (S); no longer Q3.2 (D)
- net Vicor_In: now also Q4.3 (S); no longer Q4.2 (D)
Other:
- moved on the sheet: Q3, Q4
Changed lines of the file:
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@@
   (junction (at 140.208 94.234) (diameter 0) (color 0 0 0 0)
   )
-  (junction (at 47.498 139.7) (diameter 0) (color 0 0 0 0)
-  )
   (junction (at 182.88 122.682) (diameter 0) (color 0 0 0 0)
   )
@@
   )
   (junction (at 237.744 122.682) (diameter 0) (color 0 0 0 0)
-  )
-  (junction (at 65.532 119.126) (diameter 0) (color 0 0 0 0)
   )
   (junction (at 253.492 122.682) (diameter 0) (color 0 0 0 0)
@@
     (stroke (width 0) (type default))
   )
-  (wire (pts (xy 36.068 119.126) (xy 42.418 119.126))
+  (wire (pts (xy 47.498 144.018) (xy 47.498 139.7))
     (stroke (width 0) (type default))
   )
@@
     (stroke (width 0) (type default))
   )
-  (wire (pts (xy 52.578 119.126) (xy 65.532 119.126))
-    (stroke (width 0) (type default))
-  )
   (wire (pts (xy 145.796 146.812) (xy 145.796 94.234))
     (stroke (width 0) (type default))
@@
     (stroke (width 0) (type default))
   )
-  (wire (pts (xy 47.498 134.366) (xy 47.498 139.7))
-    (stroke (width 0) (type default))
-  )
   (wire (pts (xy 122.428 146.812) (xy 133.35 146.812))
     (stroke (width 0) (type default))
@@
     (stroke (width 0) (type default))
   )
-  (wire (pts (xy 36.068 122.174) (xy 35.814 122.174))
-    (stroke (width 0) (type default))
-  )
   (wire (pts (xy 253.492 122.682) (xy 237.744 122.682))
     (stroke (width 0) (type default))
@@
     (stroke (width 0) (type default))
   )
+  (wire (pts (xy 47.498 139.7) (xy 55.372 139.7))
+    (stroke (width 0) (type default))
+  )
   (wire (pts (xy 108.966 120.142) (xy 108.966 129.794))
     (stroke (width 0) (type default))
@@
     (stroke (width 0) (type default))
   )
-  (wire (pts (xy 47.498 139.7) (xy 47.498 144.018))
-    (stroke (width 0) (type default))
-  )
   (wire (pts (xy 129.286 115.062) (xy 129.286 117.602))
     (stroke (width 0) (type default))
@@
     (stroke (width 0) (type default))
   )
-  (wire (pts (xy 35.814 122.174) (xy 35.814 139.7))
-    (stroke (width 0) (type default))
-  )
   (wire (pts (xy 65.532 119.126) (xy 65.532 139.7))
     (stroke (width 0) (type default))
   )
-  (wire (pts (xy 47.498 139.7) (xy 55.372 139.7))
-    (stroke (width 0) (type default))
-  )
   (wire (pts (xy 203.2 78.994) (xy 208.534 78.994))
     (stroke (width 0) (type default))
@@
     (stroke (width 0) (type default))
   )
-  (wire (pts (xy 35.814 139.7) (xy 47.498 139.7))
-    (stroke (width 0) (type default))
-  )
   (wire (pts (xy 133.35 152.908) (xy 133.35 146.812))
     (stroke (width 0) (type default))
@@
     (stroke (width 0) (type default))
   )
-  (wire (pts (xy 36.068 122.174) (xy 36.068 119.126))
-    (stroke (width 0) (type default))
-  )
   (wire (pts (xy 60.198 103.886) (xy 64.262 103.886))
     (stroke (width 0) (type default))
@@
     (stroke (width 0) (type default))
   )
+  (wire (pts (xy 114.046 100.584) (xy 116.586 100.584))
+    (stroke (width 0) (type default))
+  )
   (wire (pts (xy 107.188 115.062) (xy 108.966 115.062))
     (stroke (width 0) (type default))
@@
   )
   (wire (pts (xy 122.428 167.64) (xy 115.824 167.64))
+    (stroke (width 0) (type default))
+  )
+  (wire (pts (xy 105.664 153.162) (xy 108.204 153.162))
     (stroke (width 0) (type default))
   )
@@
     )
   )
-  (symbol (lib_id "PCM_Transistor_MOSFET_AKL:IXFH34N65X2") (at 115.316 96.774 90) (unit 1)
-    (in_bom yes) (on_board yes) (dnp no) (fields_autoplaced)
+  (symbol (lib_id "PCM_Transistor_MOSFET_AKL:IXFH34N65X2") (at 115.316 96.774 270) (mirror x) (unit 1)
+    (in_bom yes) (on_board yes) (dnp no)
     (property "Reference" "Q4" (at 115.316 87.884 90)
       (effects (font (size 1.27 1.27)))
@@
       (effects (font (size 1.27 1.27)))
     )
-    (property "Footprint" "PCM_Package_TO_SOT_THT_AKL:TO-247-3_Vertical_GDS" (at 112.776 91.694 0)
+    (property "Footprint" "PCM_Package_TO_SOT_THT_AKL:TO-247-3_Vertical_GDS" (at 117.856 91.694 0)
       (effects (font (size 1.27 1.27)) hide)
     )
@@
         (path "/e63e39d7-6ac0-4ffd-8aa3-1841a4541b55/9c1412ff-15e3-4ef7-9c9c-e6f8f725cc08"
           (reference "U4") (unit 1)
-        )
-      )
-    )
-  )
-  (symbol (lib_id "PCM_Transistor_BJT_AKL:MMBT2222") (at 47.498 121.666 270) (mirror x) (unit 1)
-    (in_bom yes) (on_board yes) (dnp no)
-    (property "Reference" "Q6" (at 47.498 112.776 90)
-      (effects (font (size 1.27 1.27)))
-    )
-    (property "Value" "MMBT2222" (at 47.498 115.316 90)
-      (effects (font (size 1.27 1.27)))
-    )
-    (property "Footprint" "Package_TO_SOT_SMD:SOT-23" (at 50.038 116.586 0)
-      (effects (font (size 1.27 1.27)) hide)
-    )
-    (property "Datasheet" "https://www.tme.eu/Document/fd53f7282772c4b53c43aa6dcf874bac/mmbt2222.pdf" (at 47.498 121.666 0)
-      (effects (font (size 1.27 1.27)) hide)
-    )
-    (pin "1")
-    (pin "2")
-    (pin "3")
-    (instances
-      (project "Big Daddy"
-        (path "/e63e39d7-6ac0-4ffd-8aa3-1841a4541b55/9c1412ff-15e3-4ef7-9c9c-e6f8f725cc08"
-          (reference "Q6") (unit 1)
         )
       )
@@
     )
   )
-  (symbol (lib_id "PCM_Transistor_MOSFET_AKL:IXFH34N65X2") (at 106.934 149.352 90) (unit 1)
-    (in_bom yes) (on_board yes) (dnp no) (fields_autoplaced)
+  (symbol (lib_id "PCM_Transistor_MOSFET_AKL:IXFH34N65X2") (at 106.934 149.352 270) (mirror x) (unit 1)
+    (in_bom yes) (on_board yes) (dnp no)
     (property "Reference" "Q3" (at 106.934 140.462 90)
       (effects (font (size 1.27 1.27)))
@@
       (effects (font (size 1.27 1.27)))
     )
-    (property "Footprint" "PCM_Package_TO_SOT_THT_AKL:TO-247-3_Vertical_GDS" (at 104.394 144.272 0)
+    (property "Footprint" "PCM_Package_TO_SOT_THT_AKL:TO-247-3_Vertical_GDS" (at 109.474 144.272 0)
       (effects (font (size 1.27 1.27)) hide)
     )
@@
         )
       )
-    )
-  )
-  (symbol (lib_id "Device:R_US") (at 47.498 130.556 0) (unit 1)
-    (in_bom yes) (on_board yes) (dnp no) (fields_autoplaced)
-    (property "Reference" "R41" (at 50.292 129.286 0)
-      (effects (font (size 1.27 1.27)) (justify left))
-    )
-    (property "Value" "100" (at 50.292 131.826 0)
-      (effects (font (size 1.27 1.27)) (justify left))
-    )
-    (property "Footprint" "Resistor_SMD:R_0603_1608Metric_Pad0.98x0.95mm_HandSolder" (at 48.514 130.81 90)
-      (effects (font (size 1.27 1.27)) hide)
-    )
-    (property "Datasheet" "~" (at 47.498 130.556 0)
-      (effects (font (size 1.27 1.27)) hide)
-    )
-    (pin "1")
-    (pin "2")
-    (instances
-      (project "Big Daddy"
-        (path "/e63e39d7-6ac0-4ffd-8aa3-1841a4541b55/9c1412ff-15e3-4ef7-9c9c-e6f8f725cc08"
-          (reference "R41") (unit 1)
-        )
-      )

Commit message: George Redlines for Big Daddy board
Other:
- note added: "Check datasheet for output cap suggestion, Up to 4 47uF caps recommended."
- note added: "Strange net line with a loop? Change to a straight connection"
- note added: "You probably have values for these caps. Add cap values to schematic"
Changed lines of the file:
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@@
     (fill (type none))
+  )
+  (arc (start 106.68 113.03) (mid 98.1593 94.2429) (end 105.41 74.93)
+    (stroke (width 0) (type default) (color 255 12 84 1))
+    (fill (type none))
+  )
+  (text "Strange net line with a loop?\nChange to a straight connection"
+    (at 97.79 74.93 0)
+    (effects (font (size 1.27 1.27) (color 255 3 49 1)) (justify left bottom))
+  )
+  (text "You probably have values for these caps.\nAdd cap values to schematic"
+    (at 30.48 171.45 0)
+    (effects (font (size 1.27 1.27) (color 255 3 49 1)) (justify left bottom))
   )
   (text "Fusing" (at 212.09 26.924 0)
     (effects (font (size 3 3)) (justify left bottom))
   )
+  (text "Check datasheet for output cap suggestion,\nUp to 4 47uF caps recommended. "
+    (at 218.44 154.94 0)
+    (effects (font (size 1.27 1.27) (color 255 8 4 1)) (justify left bottom))
+  )
   (text "Power Regulation" (at 234.188 112.522 0)
     (effects (font (size 3 3)) (justify right bottom))
@@
   (symbol (lib_name "LT1528CQ#PBF_1") (lib_id "LT1528CQ#PBF:LT1528CQ#PBF") (at 200.66 122.682 0) (unit 1)
     (in_bom yes) (on_board yes) (dnp no) (fields_autoplaced)
-    (property "Reference" "U4" (at 217.17 115.2144 0)
-      (effects (font (size 1.27 1.27)))
-    )
-    (property "Value" "LT1528CQ#PBF" (at 217.17 117.7544 0)
-      (effects (font (size 1.27 1.27)))
-    )
+    (property "Reference" "U4" (at 217.17 115.57 0)
+      (effects (font (size 1.27 1.27)))
+    )
+    (property "Value" "LT1528CQ#PBF" (at 217.17 118.11 0)
+      (effects (font (size 1.27 1.27)))
+    )
