File: Big Daddy/Fusing.kicad_sch (KiCad schematic)
At the start: 30 parts, among them K1 T9VV1K15-12S, Q3 IXFH34N65X2, Q4 IXFH34N65X2, U11 LM5050-1, U12 LM5050-1, U14 LM317_TO-263, U4 LT1528CQ#PBF

Commit message: Updated BOM
Parts:
- C18, C19, C20: value C -> .1uF; Digikey part number (none) -> 311-1088-1-ND; Manufacturer_Part_Number (none) -> CC0603KRX7R7BB104
- C4: value 10uf -> 10uF; Digikey part number (none) -> 1276-1038-1-ND; Manufacturer_Part_Number (none) -> CL10A106KQ8NNNC
- C5: Digikey part number (none) -> 1276-1274-1-ND; Manufacturer_Part_Number (none) -> CL10A226MP8NUNE
- D10, D11: Digikey part number (none) -> SS16T3GOSCT-ND; Manufacturer_Part_Number (none) -> SS16T3G
- D2: Digikey part number (none) -> 1655-1N4148WCT-ND; Manufacturer_Part_Number (none) -> 1N4148W
- D3: Digikey part number (none) -> 1801-TS4148RCGCT-ND; Manufacturer_Part_Number (none) -> TS4148 RCG
- K1: Digikey part number (none) -> PB2352-ND; Manufacturer_Part_Number (none) -> T9VV1K15-12S
- R17: Digikey part number (none) -> 2019-WK73R1JTTD331JCT-ND; Manufacturer_Part_Number (none) -> WK73R1JTTD331J
- R34: Digikey part number (none) -> P19315CT-ND; Manufacturer_Part_Number (none) -> ERJ-6DSFR20V
- R42: Digikey part number (none) -> 311-2.4KGRCT-ND; Manufacturer_Part_Number (none) -> RC0603JR-072K4L
- R43: Digikey part number (none) -> 541-5280-1-ND; Manufacturer_Part_Number (none) -> CRCW0603240RFKEAC
- U4: Digikey part number (none) -> LT1528CQ#PBF-ND
Connections:
- net 12_prefuse: now also Q3.3 (S), Q4.3 (S); no longer Q3.2 (D), Q4.2 (D)
- net Batt_12_IN: now also Q3.2 (D); no longer Q3.3 (S)
- net Vicor_In: now also Q4.2 (D); no longer Q4.3 (S)
Other:
- moved on the sheet: Q3, Q4
