File: Big Daddy/Latching.kicad_sch (KiCad schematic)
At the start: 12 parts, among them J1 BMS Button, J2 IMD Button, K2 G5V-2, K3 G5V-2

Commit message: George Redlines for Big Daddy board
Other:
- note added: "Assuming K2 and K3 are the "G5V-2-DC12" version of the relay. Specify full part number."
Changed lines of the file:
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@@
     (effects (font (size 1.27 1.27)) (justify left bottom))
+  )
+  (text "Assuming K2 and K3 are the \"G5V-2-DC12\" version\nof the relay. Specify full part number."
+    (at 31.75 22.86 0)
+    (effects (font (size 1.27 1.27) (color 255 2 4 1)) (justify left bottom))
   )
   (text "Pulled Low, \nHigh when no fault" (at 149.6568 113.5634 0)
