File: Big Daddy/Latching.kicad_sch (KiCad schematic)
At the start: 12 parts, among them J1 JST-B2B-VERT-2PIN, J2 JST-B2B-VERT-2PIN, K2 G5V-2, K3 G5V-2

Commit message: post comp
Parts:
- J1: value JST-B2B-VERT-2PIN -> BMS Button
- J2: value JST-B2B-VERT-2PIN -> IMD Button
Changed lines of the file:
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@@
       (effects (font (size 1.27 1.27)) (justify right))
     )
-    (property "Value" "JST-B2B-VERT-2PIN" (at 163.576 90.805 90)
+    (property "Value" "IMD Button" (at 159.766 90.805 90)
       (effects (font (size 1.27 1.27)) (justify right))
     )
@@
       (effects (font (size 1.27 1.27)) (justify right))
     )
-    (property "Value" "JST-B2B-VERT-2PIN" (at 136.017 90.17 90)
+    (property "Value" "BMS Button" (at 129.921 90.297 90)
       (effects (font (size 1.27 1.27)) (justify right))
     )

Commit message: Updated BOM
Parts:
- D5, D6: value 1N4148 -> 1N4148W; Digikey part number (none) -> 1655-1N4148WCT-ND; Manufacturer_Part_Number (none) -> 1N4148W
- R18, R23: Digikey part number (none) -> 2019-RK73H1JTTD1002FCT-ND; Manufacturer_Part_Number (none) -> RK73H1JTTD1002F
- R19, R21: value 6k -> 5.97k; Digikey part number (none) -> 2019-RN73R1JTTD5971B25CT-ND; Manufacturer_Part_Number (none) -> RN73R1JTTD5971B25
- R20, R22: Digikey part number (none) -> A129692CT-ND; Manufacturer_Part_Number (none) -> CRGCQ0603F2K2
Other:
- note added: "go to ligts on dash via microcontroller"
- note added: "safety relay"
