File: Big Daddy/Micro.kicad_sch (KiCad schematic)
At the start: 25 parts, among them Q1 2N7002, U1 MAX33054EASA+T, U2 ESP32-S3-DevKitC, U3 ESP32-S3-DevKitC

Commit message: George Redlines for Big Daddy board
Other:
- note added: "Add a decoupling cap to input"
- note added: "Instead of using "VDD", suggest using the voltage value "3.3V"."
- note added: "Note: Careful on GPIO current source. I believe the dev board has ~250mA available. LEDs, transistor and relays and maybe more?"
Changed lines of the file:
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@@
     (stroke (width 0) (type default))
+  )
+  (text "Add a decoupling cap to input" (at 161.29 46.99 0)
+    (effects (font (size 1.27 1.27) (color 255 1 57 1)) (justify left bottom))
   )
   (text "CAN Transceiver" (at 42.545 147.32 0)
     (effects (font (size 3 3)) (justify left bottom))
   )
+  (text "Note: Careful on GPIO current source. I believe the dev\n      board has ~250mA available. LEDs, transistor and \n      relays and maybe more?"
+    (at 15.24 21.59 0)
+    (effects (font (size 1.27 1.27) (color 255 0 39 1)) (justify left bottom))
+  )
+  (text "Add a decoupling cap to input" (at 77.47 48.26 0)
+    (effects (font (size 1.27 1.27) (color 255 1 57 1)) (justify left bottom))
+  )
+  (text "Instead of using \"VDD\", suggest using\nthe voltage value \"3.3V\". "
+    (at 31.75 46.99 0)
+    (effects (font (size 1.27 1.27) (color 255 0 42 1)) (justify left bottom))
+  )
   (text "Buzzer Output" (at 116.84 161.29 0)
