File: Big Daddy/TSAL.kicad_sch (KiCad schematic)
At the start: 19 parts, among them Q2 BCP53, U5 LTV-817S, U6 ICM7555xB, U7 IS31LT3360

Commit message: George Redlines for Big Daddy board
Other:
- note added: "Best Practice: Avoid 4 connections at one junction. Keep junctions to <=3 connections. Offset connections to keep <4 connections. ("T" connections instead of "+" connections) --General note for entire schematic --"
Changed lines of the file:
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@@
+    (fill (type none))
+  )
+  (arc (start 137.16 72.39) (mid 158.3065 48.0079) (end 190.5 45.72)
+    (stroke (width 0) (type default) (color 255 10 37 1))
+    (fill (type none))
+  )
+  (arc (start 198.12 91.44) (mid 185.7391 70.5301) (end 191.77 46.99)
+    (stroke (width 0) (type default) (color 255 12 14 1))
     (fill (type none))
   )
@@
     (stroke (width 0) (type default))
     (fill (type none))
+  )
+  (text "Best Practice: Avoid 4 connections at one\njunction. Keep junctions to <=3 connections.\nOffset connections to keep <4 connections.\n(\"T\" connections instead of \"+\" connections)\n--General note for entire schematic --"
+    (at 191.77 43.18 0)
+    (effects (font (size 1.27 1.27) (color 255 0 54 1)) (justify left bottom))
   )
   (text "*Optional just in case LED Drive does not work" (at 189.484 128.016 0)
@@
           (reference "R24") (unit 1)
         )
-        (path "/e63e39d7-6ac0-4ffd-8aa3-1841a4541b55/86dc982f-3c1c-4a60-9b44-a3fbe3fd622a/edff7200-18c6-4e0c-99f9-a118fc24b63a"
-          (reference "R34") (unit 1)
-        )
-      )
+      )
