File: Big Daddy/TSAL.kicad_sch (KiCad schematic)
At the start: 19 parts, among them Q2 BCP53, U5 LTV-817S, U6 ICM7555xB, U7 IS31LT3360

Commit message: so cloes
Connections:
- net VCC renamed VDD
Changed lines of the file:
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@@
     (stroke (width 0) (type default))
   )
-  (wire (pts (xy 157.48 70.612) (xy 134.366 70.612))
+  (wire (pts (xy 134.366 70.612) (xy 157.48 70.612))
+    (stroke (width 0) (type default))
+  )
+  (wire (pts (xy 77.216 101.854) (xy 77.216 102.108))
     (stroke (width 0) (type default))
   )
@@
     (stroke (width 0) (type default))
   )
-  (wire (pts (xy 134.366 68.326) (xy 134.366 70.612))
+  (wire (pts (xy 134.366 68.58) (xy 134.366 70.612))
     (stroke (width 0) (type default))
   )
@@
     (stroke (width 0) (type default))
   )
+  (wire (pts (xy 72.898 102.108) (xy 77.216 102.108))
+    (stroke (width 0) (type default))
+  )
   (wire (pts (xy 147.066 99.314) (xy 160.274 99.314))
     (stroke (width 0) (type default))
@@
   )
   (wire (pts (xy 207.772 79.756) (xy 215.9 79.756))
-    (stroke (width 0) (type default))
-  )
-  (wire (pts (xy 72.898 102.108) (xy 78.486 102.108))
     (stroke (width 0) (type default))
   )
@@
     )
   )
-  (symbol (lib_id "power:VCC") (at 134.366 68.326 0) (unit 1)
-    (in_bom yes) (on_board yes) (dnp no) (fields_autoplaced)
-    (property "Reference" "#PWR040" (at 134.366 72.136 0)
-      (effects (font (size 1.27 1.27)) hide)
-    )
-    (property "Value" "VCC" (at 134.366 63.5 0)
-      (effects (font (size 1.27 1.27)))
-    )
-    (property "Footprint" "" (at 134.366 68.326 0)
-      (effects (font (size 1.27 1.27)) hide)
-    )
-    (property "Datasheet" "" (at 134.366 68.326 0)
-      (effects (font (size 1.27 1.27)) hide)
-    )
-    (pin "1")
-    (instances
-      (project "Big Daddy"
-        (path "/e63e39d7-6ac0-4ffd-8aa3-1841a4541b55/86dc982f-3c1c-4a60-9b44-a3fbe3fd622a/7a2f50f6-0c99-4e8d-9c2a-8f2f961d2e6d"
-          (reference "#PWR040") (unit 1)
-        )
-      )
-    )
-  )
   (symbol (lib_id "Device:R_US") (at 160.274 91.694 0) (unit 1)
     (in_bom yes) (on_board yes) (dnp no) (fields_autoplaced)
@@
         (path "/e63e39d7-6ac0-4ffd-8aa3-1841a4541b55/86dc982f-3c1c-4a60-9b44-a3fbe3fd622a/7a2f50f6-0c99-4e8d-9c2a-8f2f961d2e6d"
           (reference "#PWR045") (unit 1)
+        )
+      )
+    )
+  )
+  (symbol (lib_id "power:VDD") (at 134.366 68.58 0) (unit 1)
+    (in_bom yes) (on_board yes) (dnp no) (fields_autoplaced)
+    (property "Reference" "#PWR059" (at 134.366 72.39 0)
+      (effects (font (size 1.27 1.27)) hide)
+    )
+    (property "Value" "VDD" (at 134.366 63.246 0)
+      (effects (font (size 1.27 1.27)))
+    )
+    (property "Footprint" "" (at 134.366 68.58 0)
+      (effects (font (size 1.27 1.27)) hide)
+    )
+    (property "Datasheet" "" (at 134.366 68.58 0)
+      (effects (font (size 1.27 1.27)) hide)
+    )
+    (pin "1")
+    (instances
+      (project "Big Daddy"
+        (path "/e63e39d7-6ac0-4ffd-8aa3-1841a4541b55/86dc982f-3c1c-4a60-9b44-a3fbe3fd622a/7a2f50f6-0c99-4e8d-9c2a-8f2f961d2e6d"
+          (reference "#PWR059") (unit 1)
         )
       )
@@
         (path "/e63e39d7-6ac0-4ffd-8aa3-1841a4541b55/86dc982f-3c1c-4a60-9b44-a3fbe3fd622a/7a2f50f6-0c99-4e8d-9c2a-8f2f961d2e6d"
           (reference "R26") (unit 1)
-        )
-      )
-    )
-  )
-  (symbol (lib_id "power:VCC") (at 78.486 102.108 0) (unit 1)
-    (in_bom yes) (on_board yes) (dnp no) (fields_autoplaced)
-    (property "Reference" "#PWR037" (at 78.486 105.918 0)
-      (effects (font (size 1.27 1.27)) hide)
-    )
-    (property "Value" "VCC" (at 78.486 97.282 0)
-      (effects (font (size 1.27 1.27)))
-    )
-    (property "Footprint" "" (at 78.486 102.108 0)
-      (effects (font (size 1.27 1.27)) hide)
-    )
-    (property "Datasheet" "" (at 78.486 102.108 0)
-      (effects (font (size 1.27 1.27)) hide)
-    )
-    (pin "1")
-    (instances
-      (project "Big Daddy"
-        (path "/e63e39d7-6ac0-4ffd-8aa3-1841a4541b55/86dc982f-3c1c-4a60-9b44-a3fbe3fd622a/7a2f50f6-0c99-4e8d-9c2a-8f2f961d2e6d"
-          (reference "#PWR037") (unit 1)
         )
       )
@@
         )
       )
+    )
+  )
+  (symbol (lib_id "power:VDD") (at 77.216 101.854 0) (unit 1)
+    (in_bom yes) (on_board yes) (dnp no) (fields_autoplaced)
+    (property "Reference" "#PWR050" (at 77.216 105.664 0)
+      (effects (font (size 1.27 1.27)) hide)
+    )
+    (property "Value" "VDD" (at 77.216 96.52 0)
+      (effects (font (size 1.27 1.27)))
+    )
+    (property "Footprint" "" (at 77.216 101.854 0)
+      (effects (font (size 1.27 1.27)) hide)
+    )
+    (property "Datasheet" "" (at 77.216 101.854 0)
+      (effects (font (size 1.27 1.27)) hide)
+    )
+    (pin "1")
+    (instances
+      (project "Big Daddy"
+        (path "/e63e39d7-6ac0-4ffd-8aa3-1841a4541b55/86dc982f-3c1c-4a60-9b44-a3fbe3fd622a/7a2f50f6-0c99-4e8d-9c2a-8f2f961d2e6d"
+          (reference "#PWR050") (unit 1)
+        )
+      )

Commit message: Updated BOM
Parts:
- C10, C9: value 0.1u -> .1uF; Digikey part number (none) -> 311-1088-1-ND; Manufacturer_Part_Number (none) -> CC0603KRX7R7BB104
- C11: value 10u -> 10uF; Digikey part number (none) -> 1276-1038-1-ND; Manufacturer_Part_Number (none) -> CL10A106KQ8NNNC
- C13: Digikey part number (none) -> 311-1088-1-ND; Manufacturer_Part_Number (none) -> CC0603KRX7R7BB104
- D9: Digikey part number (none) -> MMSZ5231B-FDICT-ND; Manufacturer_Part_Number (none) -> MMSZ5231B-7-F
- L1: Digikey part number (none) -> 587-1716-1-ND; Manufacturer_Part_Number (none) -> LBMF1608T470K
- Q2: Digikey part number (none) -> BCP53FSCT-ND; Manufacturer_Part_Number (none) -> BCP53
- R24: Digikey part number (none) -> CF12JT39K0CT-ND; Manufacturer_Part_Number (none) -> CF12JT39K0
- R25, R26, R29: Digikey part number (none) -> 2019-RK73H1JTTD1002FCT-ND; Manufacturer_Part_Number (none) -> RK73H1JTTD1002F
- R27: Digikey part number (none) -> P15KDBCT-ND; Manufacturer_Part_Number (none) -> ERA-3AEB153V
- R28: Digikey part number (none) -> RMCF0603FT1K00CT-ND; Manufacturer_Part_Number (none) -> RMCF0603FT1K00
- R30: Digikey part number (none) -> 311-.15QCT-ND; Manufacturer_Part_Number (none) -> RL0603FR-070R15L
- R31: Digikey part number (none) -> P100FCT-ND; Manufacturer_Part_Number (none) -> ERJ-8ENF1000V
- U5: Digikey part number (none) -> 160-1367-5-ND; Manufacturer_Part_Number (none) -> LTV-817S
- U6: Digikey part number (none) -> ICM7555CBAZ-TCT-ND; Manufacturer_Part_Number (none) -> ICM7555CBAZ-T
- U7: Digikey part number (none) -> 2521-IS31LT3360-SDLS4-TRCT-ND; Manufacturer_Part_Number (none) -> IS31LT3360-SDLS4-TR
