File: Big Daddy/Connectors.kicad_sch (KiCad schematic)
At the start: 6 parts, among them J10 Conn_01x02, J11 Conn_01x23, J12 Conn_01x14, J13 Conn_01x14, J8 Conn_01x14, J9 Conn_01x08

Commit message: so cloes
Parts:
- J9: footprint AMP_seal:TE_1-776280-1_8pin_Horizontal -> AERO_Footprints:TE_1-776280-1_8pin_Horizontal
Connections:
- net FAN_LED is gone; now on net RTD_LED: J12.6 (Pin_6)
- net BL_STRAIN0: now also J11.19 (Pin_19); no longer J11.23 (Pin_23)
- net BL_TEMP: now also J11.23 (Pin_23); no longer J11.19 (Pin_19)
- net BMS_12V: now also J8.4 (Pin_4); no longer J8.7 (Pin_7)
- net BMS_Fault_ind: now also J12.8 (Pin_8); no longer J12.9 (Pin_9)
- net BRAKE_PWR_OUT: now also J8.10 (Pin_10); no longer J8.5 (Pin_5)
- net BRB_LOOP: now also J9.3 (Pin_3); no longer J9.8 (Pin_8)
- net Brake_Regen: now also J12.13 (Pin_13); no longer J12.14 (Pin_14)
- net CAN_H: now also J12.2 (Pin_2); no longer J12.3 (Pin_3)
- net CAN_L: now also J12.1 (Pin_1); no longer J12.2 (Pin_2)
- net Coast_Regen: now also J12.14 (Pin_14); no longer J12.13 (Pin_13)
- net DRIVE_MODE_BTTN: now also J12.5 (Pin_5); no longer J12.11 (Pin_11)
- net DRIVE_MODE_LED: now also J12.4 (Pin_4); no longer J12.10 (Pin_10)
- net FAN_PWR_OUT: now also J8.1 (Pin_1), J8.6 (Pin_6); no longer J8.4 (Pin_4)
- net IMD_FAULT_SIG: now also J9.8 (Pin_8); no longer J9.5 (Pin_5)
- net IMD_Fault_ind: now also J12.9 (Pin_9); no longer J12.8 (Pin_8)
- net PUMP_12V: now also J8.2 (Pin_2)
- net RINE_12V: now also J8.5 (Pin_5); no longer J8.6 (Pin_6)
- net RTD_BUZZER_OUT: now also J12.10 (Pin_10); no longer J12.1 (Pin_1)
- net RTD_LED: no longer J12.5 (Pin_5)
- net SSOK: now also J9.4 (Pin_4); no longer J9.3 (Pin_3)
- net START_BTTN: now also J12.3 (Pin_3); no longer J12.12 (Pin_12)
- net TSAL_GND: now also J9.2 (Pin_2); no longer J9.1 (Pin_1)
- net TSAL_PWR: now also J9.1 (Pin_1); no longer J9.2 (Pin_2)
- net TSV: now also J9.5 (Pin_5); no longer J9.4 (Pin_4)
- net Batt_12 renamed Batt_12_IN
- net PUMP_LED: no longer names the net of J12.7 (Pin_7)

Commit message: REVIEW TIME
Connections:
- net BL_SPEED: now also J11.23 (Pin_23); no longer J11.20 (Pin_20)
- net BL_STRAIN0: now also J13.11 (Pin_11); no longer J11.19 (Pin_19)
- net BL_STRAIN1: now also J13.4 (Pin_4); no longer J11.22 (Pin_22)
- net BL_SUS: now also J11.7 (Pin_7); no longer J11.18 (Pin_18)
- net BL_TEMP: now also J11.8 (Pin_8); no longer J11.23 (Pin_23)
- net BR_SPEED: now also J11.22 (Pin_22); no longer J11.21 (Pin_21)
- net BR_STRAIN0: now also J11.19 (Pin_19); no longer J11.16 (Pin_16)
- net BR_STRAIN1: now also J11.13 (Pin_13); no longer J11.17 (Pin_17)
- net BR_SUS: now also J11.4 (Pin_4); no longer J11.14 (Pin_14)
- net BR_TEMP: now also J11.5 (Pin_5); no longer J11.15 (Pin_15)
- net FBrake: now also J13.3 (Pin_3); no longer J11.2 (Pin_2)
- net FL_SPEED: now also J11.15 (Pin_15); no longer J11.11 (Pin_11)
- net FL_STRAIN0: now also J11.10 (Pin_10); no longer J11.12 (Pin_12)
- net FL_STRAIN1: now also J11.18 (Pin_18); no longer J11.13 (Pin_13)
- net FL_SUS: now also J11.17 (Pin_17); no longer J11.9 (Pin_9)
- net FL_TEMP: now also J11.2 (Pin_2); no longer J11.10 (Pin_10)
- net FR_SPEED: now also J11.21 (Pin_21); no longer J11.6 (Pin_6)
- net FR_STRAIN0: now also J11.9 (Pin_9); no longer J11.7 (Pin_7)
- net FR_STRAIN1: now also J11.1 (Pin_1); no longer J11.8 (Pin_8)
- net FR_SUS: now also J11.16 (Pin_16); no longer J11.5 (Pin_5)
- net FR_TEMP: now also J11.14 (Pin_14); no longer J11.4 (Pin_4)
- net GPS_RX: now also J13.12 (Pin_12); no longer J13.10 (Pin_10)
- net GPS_TX: now also J13.8 (Pin_8); no longer J13.11 (Pin_11)
- net IMU_RX: now also J13.9 (Pin_9); no longer J13.8 (Pin_8)
- net IMU_TX: now also J13.5 (Pin_5); no longer J13.9 (Pin_9)
- net LoRa_RX: now also J13.14 (Pin_14); no longer J13.6 (Pin_6)
- net LoRa_TX: now also J13.13 (Pin_13); no longer J13.7 (Pin_7)
- net PUMP_TEMP_IN: now also J13.1 (Pin_1); no longer J13.14 (Pin_14)
- net PUMP_TEMP_OUT: now also J13.6 (Pin_6); no longer J13.13 (Pin_13)
- net Pedal_1: now also J13.10 (Pin_10); no longer J13.3 (Pin_3)
- net RBrake: now also J13.7 (Pin_7); no longer J11.3 (Pin_3)
- net RPi_RX: now also J11.12 (Pin_12); no longer J13.4 (Pin_4)
- net RPi_TX: now also J11.11 (Pin_11); no longer J13.5 (Pin_5)
- net STEERING: now also J11.6 (Pin_6); no longer J13.12 (Pin_12)
Changed lines of the file:
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@@
     (effects (font (size 3 3)) (justify left bottom))
   )
-  (hierarchical_label "BR_STRAIN0" (shape input) (at 109.22 93.726 0) (fields_autoplaced)
+  (hierarchical_label "BR_STRAIN0" (shape input) (at 109.22 86.106 0) (fields_autoplaced)
     (effects (font (size 1.27 1.27)) (justify left))
   )
@@
     (effects (font (size 1.27 1.27)) (justify left))
   )
-  (hierarchical_label "BR_TEMP" (shape input) (at 109.22 96.266 0) (fields_autoplaced)
+  (hierarchical_label "BR_TEMP" (shape input) (at 109.22 121.666 0) (fields_autoplaced)
     (effects (font (size 1.27 1.27)) (justify left))
   )
@@
     (effects (font (size 1.27 1.27)) (justify left))
   )
-  (hierarchical_label "BL_STRAIN0" (shape input) (at 109.22 86.106 0) (fields_autoplaced)
+  (hierarchical_label "BL_STRAIN0" (shape input) (at 200.914 44.196 0) (fields_autoplaced)
     (effects (font (size 1.27 1.27)) (justify left))
   )
-  (hierarchical_label "FL_TEMP" (shape input) (at 109.22 108.966 0) (fields_autoplaced)
+  (hierarchical_label "FL_TEMP" (shape input) (at 109.22 129.286 0) (fields_autoplaced)
     (effects (font (size 1.27 1.27)) (justify left))
   )
-  (hierarchical_label "FL_STRAIN1" (shape input) (at 109.22 101.346 0) (fields_autoplaced)
+  (hierarchical_label "FL_STRAIN1" (shape input) (at 109.22 88.646 0) (fields_autoplaced)
     (effects (font (size 1.27 1.27)) (justify left))
   )
@@
     (effects (font (size 1.27 1.27)) (justify left))
   )
-  (hierarchical_label "BL_SPEED" (shape input) (at 109.22 83.566 0) (fields_autoplaced)
+  (hierarchical_label "BL_SPEED" (shape input) (at 109.22 75.946 0) (fields_autoplaced)
     (effects (font (size 1.27 1.27)) (justify left))
   )
@@
     (effects (font (size 1.27 1.27)) (justify left))
   )
-  (hierarchical_label "PUMP_TEMP_OUT" (shape input) (at 200.914 39.116 0) (fields_autoplaced)
+  (hierarchical_label "PUMP_TEMP_OUT" (shape input) (at 200.914 56.896 0) (fields_autoplaced)
     (effects (font (size 1.27 1.27)) (justify left))
   )
-  (hierarchical_label "FL_SUS" (shape input) (at 109.22 111.506 0) (fields_autoplaced)
+  (hierarchical_label "FL_SUS" (shape input) (at 109.22 91.186 0) (fields_autoplaced)
     (effects (font (size 1.27 1.27)) (justify left))
   )
@@
     (effects (font (size 1.27 1.27)) (justify left))
   )
-  (hierarchical_label "BR_SUS" (shape input) (at 109.22 98.806 0) (fields_autoplaced)
+  (hierarchical_label "BR_SUS" (shape input) (at 109.22 124.206 0) (fields_autoplaced)
     (effects (font (size 1.27 1.27)) (justify left))
   )
@@
     (effects (font (size 1.27 1.27)) (justify left))
   )
-  (hierarchical_label "BR_SPEED" (shape input) (at 109.22 81.026 0) (fields_autoplaced)
+  (hierarchical_label "BR_SPEED" (shape input) (at 109.22 78.486 0) (fields_autoplaced)
     (effects (font (size 1.27 1.27)) (justify left))
   )
@@
     (effects (font (size 1.27 1.27)) (justify left))
   )
-  (hierarchical_label "FR_SUS" (shape input) (at 109.22 121.666 0) (fields_autoplaced)
+  (hierarchical_label "FR_SUS" (shape input) (at 109.22 93.726 0) (fields_autoplaced)
     (effects (font (size 1.27 1.27)) (justify left))
   )
@@
     (effects (font (size 1.27 1.27)) (justify left))
   )
-  (hierarchical_label "FR_STRAIN0" (shape input) (at 109.22 116.586 0) (fields_autoplaced)
+  (hierarchical_label "FR_STRAIN0" (shape input) (at 109.22 111.506 0) (fields_autoplaced)
     (effects (font (size 1.27 1.27)) (justify left))
   )
-  (hierarchical_label "IMU_RX" (shape input) (at 200.914 51.816 0) (fields_autoplaced)
+  (hierarchical_label "IMU_RX" (shape input) (at 200.914 49.276 0) (fields_autoplaced)
     (effects (font (size 1.27 1.27)) (justify left))
   )
@@
     (effects (font (size 1.27 1.27)) (justify left))
   )
-  (hierarchical_label "FR_STRAIN1" (shape input) (at 109.22 114.046 0) (fields_autoplaced)
+  (hierarchical_label "FR_STRAIN1" (shape input) (at 109.22 131.826 0) (fields_autoplaced)
     (effects (font (size 1.27 1.27)) (justify left))
   )
-  (hierarchical_label "BL_SUS" (shape input) (at 109.22 88.646 0) (fields_autoplaced)
+  (hierarchical_label "BL_SUS" (shape input) (at 109.22 116.586 0) (fields_autoplaced)
     (effects (font (size 1.27 1.27)) (justify left))
   )
@@
     (effects (font (size 1.27 1.27)) (justify left))
   )
-  (hierarchical_label "PUMP_TEMP_IN" (shape input) (at 200.914 36.576 0) (fields_autoplaced)
+  (hierarchical_label "PUMP_TEMP_IN" (shape input) (at 200.914 69.596 0) (fields_autoplaced)
     (effects (font (size 1.27 1.27)) (justify left))
   )
@@
     (effects (font (size 1.27 1.27)) (justify left))
   )
-  (hierarchical_label "STEERING" (shape input) (at 200.914 41.656 0) (fields_autoplaced)
+  (hierarchical_label "STEERING" (shape input) (at 109.22 119.126 0) (fields_autoplaced)
     (effects (font (size 1.27 1.27)) (justify left))
   )
@@
     (effects (font (size 1.27 1.27)) (justify left))
   )
-  (hierarchical_label "Pedal_1" (shape input) (at 200.914 64.516 0) (fields_autoplaced)
+  (hierarchical_label "Pedal_1" (shape input) (at 200.914 46.736 0) (fields_autoplaced)
     (effects (font (size 1.27 1.27)) (justify left))
   )
@@
     (effects (font (size 1.27 1.27)) (justify left))
   )
-  (hierarchical_label "GPS_TX" (shape input) (at 200.914 44.196 0) (fields_autoplaced)
+  (hierarchical_label "GPS_TX" (shape input) (at 200.914 51.816 0) (fields_autoplaced)
     (effects (font (size 1.27 1.27)) (justify left))
   )
@@
     (effects (font (size 1.27 1.27)) (justify left))
   )
-  (hierarchical_label "FBrake" (shape input) (at 109.22 129.286 0) (fields_autoplaced)
+  (hierarchical_label "FBrake" (shape input) (at 200.914 64.516 0) (fields_autoplaced)
     (effects (font (size 1.27 1.27)) (justify left))
   )
@@
     (effects (font (size 1.27 1.27)) (justify left))
   )
-  (hierarchical_label "FL_STRAIN0" (shape input) (at 109.22 103.886 0) (fields_autoplaced)
+  (hierarchical_label "FL_STRAIN0" (shape input) (at 109.22 108.966 0) (fields_autoplaced)
     (effects (font (size 1.27 1.27)) (justify left))
   )
@@
     (effects (font (size 1.27 1.27)) (justify left))
   )
-  (hierarchical_label "RPi_RX" (shape input) (at 200.914 61.976 0) (fields_autoplaced)
+  (hierarchical_label "RPi_RX" (shape input) (at 109.22 103.886 0) (fields_autoplaced)
     (effects (font (size 1.27 1.27)) (justify left))
   )
@@
     (effects (font (size 1.27 1.27)) (justify left))
   )
-  (hierarchical_label "RBrake" (shape input) (at 109.22 126.746 0) (fields_autoplaced)
+  (hierarchical_label "RBrake" (shape input) (at 200.914 54.356 0) (fields_autoplaced)
     (effects (font (size 1.27 1.27)) (justify left))
   )
-  (hierarchical_label "FL_SPEED" (shape input) (at 109.22 106.426 0) (fields_autoplaced)
+  (hierarchical_label "FL_SPEED" (shape input) (at 109.22 96.266 0) (fields_autoplaced)
     (effects (font (size 1.27 1.27)) (justify left))
   )
-  (hierarchical_label "FR_TEMP" (shape input) (at 109.22 124.206 0) (fields_autoplaced)
+  (hierarchical_label "FR_TEMP" (shape input) (at 109.22 98.806 0) (fields_autoplaced)
     (effects (font (size 1.27 1.27)) (justify left))
   )
@@
     (effects (font (size 1.27 1.27)) (justify left))
   )
-  (hierarchical_label "BL_TEMP" (shape input) (at 109.22 75.946 0) (fields_autoplaced)
+  (hierarchical_label "BL_TEMP" (shape input) (at 109.22 114.046 0) (fields_autoplaced)
     (effects (font (size 1.27 1.27)) (justify left))
   )
-  (hierarchical_label "LoRa_TX" (shape input) (at 200.914 54.356 0) (fields_autoplaced)
+  (hierarchical_label "LoRa_TX" (shape input) (at 200.914 39.116 0) (fields_autoplaced)
     (effects (font (size 1.27 1.27)) (justify left))
   )
-  (hierarchical_label "BR_STRAIN1" (shape input) (at 109.22 91.186 0) (fields_autoplaced)
+  (hierarchical_label "BR_STRAIN1" (shape input) (at 109.22 101.346 0) (fields_autoplaced)
     (effects (font (size 1.27 1.27)) (justify left))
   )
-  (hierarchical_label "LoRa_RX" (shape input) (at 200.914 56.896 0) (fields_autoplaced)
+  (hierarchical_label "LoRa_RX" (shape input) (at 200.914 36.576 0) (fields_autoplaced)
     (effects (font (size 1.27 1.27)) (justify left))
   )
@@
     (effects (font (size 1.27 1.27)) (justify left))
   )
-  (hierarchical_label "GPS_RX" (shape input) (at 200.914 46.736 0) (fields_autoplaced)
+  (hierarchical_label "GPS_RX" (shape input) (at 200.914 41.656 0) (fields_autoplaced)
     (effects (font (size 1.27 1.27)) (justify left))
   )
-  (hierarchical_label "BL_STRAIN1" (shape input) (at 109.22 78.486 0) (fields_autoplaced)
+  (hierarchical_label "BL_STRAIN1" (shape input) (at 200.914 61.976 0) (fields_autoplaced)
     (effects (font (size 1.27 1.27)) (justify left))
   )
-  (hierarchical_label "IMU_TX" (shape input) (at 200.914 49.276 0) (fields_autoplaced)
+  (hierarchical_label "IMU_TX" (shape input) (at 200.914 59.436 0) (fields_autoplaced)
     (effects (font (size 1.27 1.27)) (justify left))
   )
-  (hierarchical_label "RPi_TX" (shape input) (at 200.914 59.436 0) (fields_autoplaced)
+  (hierarchical_label "RPi_TX" (shape input) (at 109.22 106.426 0) (fields_autoplaced)
     (effects (font (size 1.27 1.27)) (justify left))
   )
-  (hierarchical_label "FR_SPEED" (shape input) (at 109.22 119.126 0) (fields_autoplaced)
+  (hierarchical_label "FR_SPEED" (shape input) (at 109.22 81.026 0) (fields_autoplaced)
     (effects (font (size 1.27 1.27)) (justify left))
   )

Commit message: updates
Parts:
- added J15: Conn_01x02, AERO_Footprints:TE_MATE-N-LOK_1-770866-x_1x02_P4.14mm_Vertical, symbol Connector_Generic:Conn_01x02
Connections:
- net FAN_PWR_OUT: no longer J8.1 (Pin_1)
- net GND: now reaches J12.11 (Pin_11)
- net GND: now also J11.20 (Pin_20), J11.3 (Pin_3), J12.12 (Pin_12), J12.7 (Pin_7), J8.7 (Pin_7), J8.8 (Pin_8), J8.9 (Pin_9), J15.1 (Pin_1), J15.2 (Pin_2)
- new net BMS_FAN_PWR_OUT: J8.1 (Pin_1)
Other:
- note added: "GND"
- moved on the sheet: J10
