File: Big Daddy/DCDC.kicad_sch (KiCad schematic)
At the start: 16 parts, among them U10 TLP184, U8 Vicor_AERO, U9 LTV-817S

Commit message: so cloes
Changed lines of the file:
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@@
-    )
-  )
-  (symbol (lib_id "power:VDD") (at 138.684 64.77 0) (unit 1)
-    (in_bom yes) (on_board yes) (dnp no)
-    (property "Reference" "#PWR04" (at 138.684 68.58 0)
-      (effects (font (size 1.27 1.27)) hide)
-    )
-    (property "Value" "VDD" (at 141.732 63.5 0)
-      (effects (font (size 1.27 1.27)))
-    )
-    (property "Footprint" "" (at 138.684 64.77 0)
-      (effects (font (size 1.27 1.27)) hide)
-    )
-    (property "Datasheet" "" (at 138.684 64.77 0)
-      (effects (font (size 1.27 1.27)) hide)
-    )
-    (pin "1")
-    (instances
-      (project "Big Daddy"
-        (path "/e63e39d7-6ac0-4ffd-8aa3-1841a4541b55/86f84094-3751-45ac-bbc5-d8f885869273"
-          (reference "#PWR04") (unit 1)
-        )
-        (path "/e63e39d7-6ac0-4ffd-8aa3-1841a4541b55/86dc982f-3c1c-4a60-9b44-a3fbe3fd622a/edff7200-18c6-4e0c-99f9-a118fc24b63a"
-          (reference "#PWR050") (unit 1)
-        )
-      )
     )
   )
@@
         )
       )
+    )
+  )
+  (symbol (lib_id "power:VDD") (at 138.684 64.77 0) (unit 1)
+    (in_bom yes) (on_board yes) (dnp no) (fields_autoplaced)
+    (property "Reference" "#PWR050" (at 138.684 68.58 0)
+      (effects (font (size 1.27 1.27)) hide)
+    )
+    (property "Value" "VDD" (at 138.684 59.436 0)
+      (effects (font (size 1.27 1.27)))
+    )
+    (property "Footprint" "" (at 138.684 64.77 0)
+      (effects (font (size 1.27 1.27)) hide)
+    )
+    (property "Datasheet" "" (at 138.684 64.77 0)
+      (effects (font (size 1.27 1.27)) hide)
+    )
+    (pin "1")
+    (instances
+      (project "Big Daddy"
+        (path "/e63e39d7-6ac0-4ffd-8aa3-1841a4541b55/86dc982f-3c1c-4a60-9b44-a3fbe3fd622a/7a2f50f6-0c99-4e8d-9c2a-8f2f961d2e6d"
+          (reference "#PWR050") (unit 1)
+        )
+        (path "/e63e39d7-6ac0-4ffd-8aa3-1841a4541b55/86dc982f-3c1c-4a60-9b44-a3fbe3fd622a/edff7200-18c6-4e0c-99f9-a118fc24b63a"
+          (reference "#PWR040") (unit 1)
+        )
+      )

Commit message: Updated BOM
Parts:
- L2: Digikey part number (none) -> 490-5112-1-ND; Manufacturer_Part_Number (none) -> LQM2HPN1R0MG0L
- L3: Digikey part number (none) -> CE201210-R15JCT-ND; Manufacturer_Part_Number (none) -> CE201210-R15J
- R35, R40: Digikey part number (none) -> 2019-RK73H1JTTD1002FCT-ND; Manufacturer_Part_Number (none) -> RK73H1JTTD1002F
- R36: Digikey part number (none) -> P300GCT-ND; Manufacturer_Part_Number (none) -> ERJ-3GEYJ301V
- R37, R38, R39: Digikey part number (none) -> RMCF0603FT1K00CT-ND; Manufacturer_Part_Number (none) -> RMCF0603FT1K00
- RV1: Digikey part number (none) -> TC33X-503ECT-ND; Manufacturer_Part_Number (none) -> TC33X-2-503E
- U10: Digikey part number (none) -> TLP184(BL-TPLSECT-ND; Manufacturer_Part_Number (none) -> TLP184(BL-TPL,SE
- U9: Digikey part number (none) -> 160-1367-5-ND; Manufacturer_Part_Number (none) -> LTV-817S
