File: Big Daddy/TSMP.kicad_sch (KiCad schematic)
At the start: 7 parts, among them J3 HV+, J4 HV-, J5 GND, J6 HV+, J7 HV-

Commit message: Updated BOM
Parts:
- R32, R33: value 10k -> 20k; footprint Resistor_THT:R_Axial_Power_L50.0mm_W9.0mm_P60.96mm -> Resistor_THT:R_Axial_DIN0309_L9.0mm_D3.2mm_P5.08mm_Vertical; Digikey part number (none) -> CF18JT20K0CT-ND; Manufacturer_Part_Number (none) -> CF18JT20K0
Other:
- moved on the sheet: J6, J7
